Commit message: update urdf

File: rofunc/simulator/assets/urdf/anymal_b_simple_description/urdf/anymal.urdf (robot description, URDF)
Before this commit: robot anymal, 21 links, 20 joints
Links:
- link LF_ADAPTER: geometry collision cylinder length=0.32125 radius=0.015; visual mesh filename=/home/ubuntu/Rofunc/rofunc/simulator/assets/urdf/anymal_b_s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 scale=0.001 0.001 0.001
- link LF_HIP: geometry collision cylinder length=0.03 radius=0.045; collision cylinder length=0.1 radius=0.08
- link LF_SHANK: geometry collision box size=0.08 0.07 0.13; visual mesh filename=/home/ubuntu/Rofunc/rofunc/simulator/assets/urdf/anymal_b_s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 scale=0.001 0.001 0.001
- link LF_THIGH: geometry collision box size=0.08 0.04 0.25; collision cylinder length=0.12 radius=0.06
- link LH_ADAPTER: geometry collision cylinder length=0.32125 radius=0.015; visual mesh filename=/home/ubuntu/Rofunc/rofunc/simulator/assets/urdf/anymal_b_s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 scale=0.001 0.001 0.001
- link LH_HIP: geometry collision cylinder length=0.03 radius=0.045; collision cylinder length=0.1 radius=0.08
- link LH_SHANK: geometry collision box size=0.08 0.07 0.13; visual mesh filename=/home/ubuntu/Rofunc/rofunc/simulator/assets/urdf/anymal_b_s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 scale=0.001 0.001 0.001
- link LH_THIGH: geometry collision box size=0.08 0.04 0.25; collision cylinder length=0.12 radius=0.06
- link RF_ADAPTER: geometry collision cylinder length=0.32125 radius=0.015; visual mesh filename=/home/ubuntu/Rofunc/rofunc/simulator/assets/urdf/anymal_b_s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 scale=0.001 0.001 0.001
- link RF_HIP: geometry collision cylinder length=0.03 radius=0.045; collision cylinder length=0.1 radius=0.08
- link RF_SHANK: geometry collision box size=0.08 0.07 0.13; visual mesh filename=/home/ubuntu/Rofunc/rofunc/simulator/assets/urdf/anymal_b_s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 scale=0.001 0.001 0.001
- link RF_THIGH: geometry collision box size=0.08 0.04 0.25; collision cylinder length=0.12 radius=0.06
- link RH_ADAPTER: geometry collision cylinder length=0.32125 radius=0.015; visual mesh filename=/home/ubuntu/Rofunc/rofunc/simulator/assets/urdf/anymal_b_s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 scale=0.001 0.001 0.001
- link RH_HIP: geometry collision cylinder length=0.03 radius=0.045; collision cylinder length=0.1 radius=0.08
- link RH_SHANK: geometry collision box size=0.08 0.07 0.13; visual mesh filename=/home/ubuntu/Rofunc/rofunc/simulator/assets/urdf/anymal_b_s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 scale=0.001 0.001 0.001
- link RH_THIGH: geometry collision box size=0.08 0.04 0.25; collision cylinder length=0.12 radius=0.06
- link base: geometry collision box size=0.1 0.1 0.07; collision box size=0.1 0.1 0.07

File: rofunc/simulator/assets/urdf/curi/urdf/curi_cartesio.urdf (robot description, URDF)
Before this commit: robot curi, 35 links, 34 joints
Links:
- link control_box: geometry collision mesh filename=/home/ubuntu/Rofunc/rofunc/simulator/assets/urdf/curi_descr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; visual mesh filename=/home/ubuntu/Rofunc/rofunc/simulator/assets/urdf/curi_descr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
- link head_base: geometry collision mesh filename=/home/ubuntu/Rofunc/rofunc/simulator/assets/urdf/curi_descr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; visual mesh filename=/home/ubuntu/Rofunc/rofunc/simulator/assets/urdf/curi_descr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
- link head_link1: geometry collision mesh filename=/home/ubuntu/Rofunc/rofunc/simulator/assets/urdf/curi_descr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; visual mesh filename=/home/ubuntu/Rofunc/rofunc/simulator/assets/urdf/curi_descr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
- link head_link2: geometry collision mesh filename=/home/ubuntu/Rofunc/rofunc/simulator/assets/urdf/curi_descr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; visual mesh filename=/home/ubuntu/Rofunc/rofunc/simulator/assets/urdf/curi_descr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
- link panda_left_hand: geometry collision mesh filename=/home/ubuntu/Rofunc/rofunc/simulator/assets/urdf/curi_descr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; visual mesh filename=/home/ubuntu/Rofunc/rofunc/simulator/assets/urdf/curi_descr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
- link panda_left_link0: geometry collision mesh filename=/home/ubuntu/Rofunc/rofunc/simulator/assets/urdf/curi_descr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; visual mesh filename=/home/ubuntu/Rofunc/rofunc/simulator/assets/urdf/curi_descr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
- link panda_left_link1: geometry collision mesh filename=/home/ubuntu/Rofunc/rofunc/simulator/assets/urdf/curi_descr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; visual mesh filename=/home/ubuntu/Rofunc/rofunc/simulator/assets/urdf/curi_descr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
- link panda_left_link2: geometry collision mesh filename=/home/ubuntu/Rofunc/rofunc/simulator/assets/urdf/curi_descr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; visual mesh filename=/home/ubuntu/Rofunc/rofunc/simulator/assets/urdf/curi_descr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
- link panda_left_link3: geometry collision mesh filename=/home/ubuntu/Rofunc/rofunc/simulator/assets/urdf/curi_descr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; visual mesh filename=/home/ubuntu/Rofunc/rofunc/simulator/assets/urdf/curi_descr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
- link panda_left_link4: geometry collision mesh filename=/home/ubuntu/Rofunc/rofunc/simulator/assets/urdf/curi_descr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; visual mesh filename=/home/ubuntu/Rofunc/rofunc/simulator/assets/urdf/curi_descr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
- link panda_left_link5: geometry collision mesh filename=/home/ubuntu/Rofunc/rofunc/simulator/assets/urdf/curi_descr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; visual mesh filename=/home/ubuntu/Rofunc/rofunc/simulator/assets/urdf/curi_descr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
- link panda_left_link6: geometry collision mesh filename=/home/ubuntu/Rofunc/rofunc/simulator/assets/urdf/curi_descr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; visual mesh filename=/home/ubuntu/Rofunc/rofunc/simulator/assets/urdf/curi_descr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
- link panda_left_link7: geometry collision mesh filename=/home/ubuntu/Rofunc/rofunc/simulator/assets/urdf/curi_descr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; visual mesh filename=/home/ubuntu/Rofunc/rofunc/simulator/assets/urdf/curi_descr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
- link panda_right_hand: geometry collision mesh filename=/home/ubuntu/Rofunc/rofunc/simulator/assets/urdf/curi_descr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; visual mesh filename=/home/ubuntu/Rofunc/rofunc/simulator/assets/urdf/curi_descr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
- link panda_right_link0: geometry collision mesh filename=/home/ubuntu/Rofunc/rofunc/simulator/assets/urdf/curi_descr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; visual mesh filename=/home/ubuntu/Rofunc/rofunc/simulator/assets/urdf/curi_descr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
- link panda_right_link1: geometry collision mesh filename=/home/ubuntu/Rofunc/rofunc/simulator/assets/urdf/curi_descr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; visual mesh filename=/home/ubuntu/Rofunc/rofunc/simulator/assets/urdf/curi_descr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
- link panda_right_link2: geometry collision mesh filename=/home/ubuntu/Rofunc/rofunc/simulator/assets/urdf/curi_descr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; visual mesh filename=/home/ubuntu/Rofunc/rofunc/simulator/assets/urdf/curi_descr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
- link panda_right_link3: geometry collision mesh filename=/home/ubuntu/Rofunc/rofunc/simulator/assets/urdf/curi_descr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; visual mesh filename=/home/ubuntu/Rofunc/rofunc/simulator/assets/urdf/curi_descr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
- link panda_right_link4: geometry collision mesh filename=/home/ubuntu/Rofunc/rofunc/simulator/assets/urdf/curi_descr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; visual mesh filename=/home/ubuntu/Rofunc/rofunc/simulator/assets/urdf/curi_descr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
- link panda_right_link5: geometry collision mesh filename=/home/ubuntu/Rofunc/rofunc/simulator/assets/urdf/curi_descr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; visual mesh filename=/home/ubuntu/Rofunc/rofunc/simulator/assets/urdf/curi_descr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
- link panda_right_link6: geometry collision mesh filename=/home/ubuntu/Rofunc/rofunc/simulator/assets/urdf/curi_descr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; visual mesh filename=/home/ubuntu/Rofunc/rofunc/simulator/assets/urdf/curi_descr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
- link panda_right_link7: geometry collision mesh filename=/home/ubuntu/Rofunc/rofunc/simulator/assets/urdf/curi_descr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; visual mesh filename=/home/ubuntu/Rofunc/rofunc/simulator/assets/urdf/curi_descr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
- link summit_xls_back_left_wheel_link: geometry collision cylinder length=0.087 radius=0.127; visual mesh filename=/home/ubuntu/Rofunc/rofunc/simulator/assets/urdf/curi_descr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
- link summit_xls_back_right_wheel_link: geometry collision cylinder length=0.087 radius=0.127; visual mesh filename=/home/ubuntu/Rofunc/rofunc/simulator/assets/urdf/curi_descr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
- link summit_xls_base_link: geometry collision mesh filename=/home/ubuntu/Rofunc/rofunc/simulator/assets/urdf/curi_descr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; visual mesh filename=/home/ubuntu/Rofunc/rofunc/simulator/assets/urdf/curi_descr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
- link summit_xls_front_left_wheel_link: geometry collision cylinder length=0.087 radius=0.127; visual mesh filename=/home/ubuntu/Rofunc/rofunc/simulator/assets/urdf/curi_descr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
- link summit_xls_front_right_wheel_link: geometry collision cylinder length=0.087 radius=0.127; visual mesh filename=/home/ubuntu/Rofunc/rofunc/simulator/assets/urdf/curi_descr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
- link torso_base1: geometry collision mesh filename=/home/ubuntu/Rofunc/rofunc/simulator/assets/urdf/curi_descr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; visual mesh filename=/home/ubuntu/Rofunc/rofunc/simulator/assets/urdf/curi_descr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
- link torso_base2: geometry collision mesh filename=/home/ubuntu/Rofunc/rofunc/simulator/assets/urdf/curi_descr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; visual mesh filename=/home/ubuntu/Rofunc/rofunc/simulator/assets/urdf/curi_descr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
- link torso_end: geometry collision mesh filename=/home/ubuntu/Rofunc/rofunc/simulator/assets/urdf/curi_descr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; visual mesh filename=/home/ubuntu/Rofunc/rofunc/simulator/assets/urdf/curi_descr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
- link torso_link_b2: geometry collision mesh filename=/home/ubuntu/Rofunc/rofunc/simulator/assets/urdf/curi_descr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; visual mesh filename=/home/ubuntu/Rofunc/rofunc/simulator/assets/urdf/curi_descr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
- link torso_link_c1: geometry collision mesh filename=/home/ubuntu/Rofunc/rofunc/simulator/assets/urdf/curi_descr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; visual mesh filename=/home/ubuntu/Rofunc/rofunc/simulator/assets/urdf/curi_descr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
- link torso_middle: geometry collision mesh filename=/home/ubuntu/Rofunc/rofunc/simulator/assets/urdf/curi_descr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; visual mesh filename=/home/ubuntu/Rofunc/rofunc/simulator/assets/urdf/curi_descr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

File: rofunc/simulator/assets/urdf/curi/urdf/curi_mujoco.urdf (robot description, URDF)
Before this commit: robot curi, 41 links, 40 joints
Links:
- link control_box: geometry collision mesh filename=/home/ubuntu/Rofunc/rofunc/simulator/assets/urdf/curi_descr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; visual mesh filename=/home/ubuntu/Rofunc/rofunc/simulator/assets/urdf/curi_descr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
- link head_base: geometry collision mesh filename=/home/ubuntu/Rofunc/rofunc/simulator/assets/urdf/curi_descr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; visual mesh filename=/home/ubuntu/Rofunc/rofunc/simulator/assets/urdf/curi_descr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
- link head_link1: geometry collision mesh filename=/home/ubuntu/Rofunc/rofunc/simulator/assets/urdf/curi_descr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; visual mesh filename=/home/ubuntu/Rofunc/rofunc/simulator/assets/urdf/curi_descr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
- link head_link2: geometry collision mesh filename=/home/ubuntu/Rofunc/rofunc/simulator/assets/urdf/curi_descr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; visual mesh filename=/home/ubuntu/Rofunc/rofunc/simulator/assets/urdf/curi_descr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
- link panda_left_hand: geometry collision mesh filename=/home/ubuntu/Rofunc/rofunc/simulator/assets/urdf/curi_descr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; visual mesh filename=/home/ubuntu/Rofunc/rofunc/simulator/assets/urdf/curi_descr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
- link panda_left_leftfinger: geometry collision box size=17.5e-3 15.2e-3 18.5e-3; collision box size=17.5e-3 7e-3 23.5e-3
- link panda_left_link0: geometry collision mesh filename=/home/ubuntu/Rofunc/rofunc/simulator/assets/urdf/curi_descr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; visual mesh filename=/home/ubuntu/Rofunc/rofunc/simulator/assets/urdf/curi_descr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
- link panda_left_link1: geometry collision mesh filename=/home/ubuntu/Rofunc/rofunc/simulator/assets/urdf/curi_descr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; visual mesh filename=/home/ubuntu/Rofunc/rofunc/simulator/assets/urdf/curi_descr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
- link panda_left_link2: geometry collision mesh filename=/home/ubuntu/Rofunc/rofunc/simulator/assets/urdf/curi_descr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; visual mesh filename=/home/ubuntu/Rofunc/rofunc/simulator/assets/urdf/curi_descr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
- link panda_left_link3: geometry collision mesh filename=/home/ubuntu/Rofunc/rofunc/simulator/assets/urdf/curi_descr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; visual mesh filename=/home/ubuntu/Rofunc/rofunc/simulator/assets/urdf/curi_descr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
- link panda_left_link4: geometry collision mesh filename=/home/ubuntu/Rofunc/rofunc/simulator/assets/urdf/curi_descr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; visual mesh filename=/home/ubuntu/Rofunc/rofunc/simulator/assets/urdf/curi_descr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
- link panda_left_link5: geometry collision mesh filename=/home/ubuntu/Rofunc/rofunc/simulator/assets/urdf/curi_descr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; visual mesh filename=/home/ubuntu/Rofunc/rofunc/simulator/assets/urdf/curi_descr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
- link panda_left_link6: geometry collision mesh filename=/home/ubuntu/Rofunc/rofunc/simulator/assets/urdf/curi_descr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; visual mesh filename=/home/ubuntu/Rofunc/rofunc/simulator/assets/urdf/curi_descr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
- link panda_left_link7: geometry collision mesh filename=/home/ubuntu/Rofunc/rofunc/simulator/assets/urdf/curi_descr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; visual mesh filename=/home/ubuntu/Rofunc/rofunc/simulator/assets/urdf/curi_descr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
- link panda_left_rightfinger: geometry collision box size=17.5e-3 15.2e-3 18.5e-3; collision box size=17.5e-3 7e-3 23.5e-3
- link panda_right_hand: geometry collision mesh filename=/home/ubuntu/Rofunc/rofunc/simulator/assets/urdf/curi_descr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; visual mesh filename=/home/ubuntu/Rofunc/rofunc/simulator/assets/urdf/curi_descr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
- link panda_right_leftfinger: geometry collision box size=17.5e-3 15.2e-3 18.5e-3; collision box size=17.5e-3 7e-3 23.5e-3
- link panda_right_link0: geometry collision mesh filename=/home/ubuntu/Rofunc/rofunc/simulator/assets/urdf/curi_descr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; visual mesh filename=/home/ubuntu/Rofunc/rofunc/simulator/assets/urdf/curi_descr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
- link panda_right_link1: geometry collision mesh filename=/home/ubuntu/Rofunc/rofunc/simulator/assets/urdf/curi_descr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; visual mesh filename=/home/ubuntu/Rofunc/rofunc/simulator/assets/urdf/curi_descr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
- link panda_right_link2: geometry collision mesh filename=/home/ubuntu/Rofunc/rofunc/simulator/assets/urdf/curi_descr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; visual mesh filename=/home/ubuntu/Rofunc/rofunc/simulator/assets/urdf/curi_descr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
- link panda_right_link3: geometry collision mesh filename=/home/ubuntu/Rofunc/rofunc/simulator/assets/urdf/curi_descr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; visual mesh filename=/home/ubuntu/Rofunc/rofunc/simulator/assets/urdf/curi_descr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
- link panda_right_link4: geometry collision mesh filename=/home/ubuntu/Rofunc/rofunc/simulator/assets/urdf/curi_descr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; visual mesh filename=/home/ubuntu/Rofunc/rofunc/simulator/assets/urdf/curi_descr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
- link panda_right_link5: geometry collision mesh filename=/home/ubuntu/Rofunc/rofunc/simulator/assets/urdf/curi_descr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; visual mesh filename=/home/ubuntu/Rofunc/rofunc/simulator/assets/urdf/curi_descr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
- link panda_right_link6: geometry collision mesh filename=/home/ubuntu/Rofunc/rofunc/simulator/assets/urdf/curi_descr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; visual mesh filename=/home/ubuntu/Rofunc/rofunc/simulator/assets/urdf/curi_descr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
- link panda_right_link7: geometry collision mesh filename=/home/ubuntu/Rofunc/rofunc/simulator/assets/urdf/curi_descr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; visual mesh filename=/home/ubuntu/Rofunc/rofunc/simulator/assets/urdf/curi_descr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
- link panda_right_rightfinger: geometry collision box size=17.5e-3 15.2e-3 18.5e-3; collision box size=17.5e-3 7e-3 23.5e-3
- link summit_xls_back_left_wheel_link: geometry collision cylinder length=0.087 radius=0.127; visual mesh filename=/home/ubuntu/Rofunc/rofunc/simulator/assets/urdf/curi_descr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
- link summit_xls_back_right_wheel_link: geometry collision cylinder length=0.087 radius=0.127; visual mesh filename=/home/ubuntu/Rofunc/rofunc/simulator/assets/urdf/curi_descr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
- link summit_xls_base_link: geometry collision mesh filename=/home/ubuntu/Rofunc/rofunc/simulator/assets/urdf/curi_descr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; visual mesh filename=/home/ubuntu/Rofunc/rofunc/simulator/assets/urdf/curi_descr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
- link summit_xls_front_left_wheel_link: geometry collision cylinder length=0.087 radius=0.127; visual mesh filename=/home/ubuntu/Rofunc/rofunc/simulator/assets/urdf/curi_descr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
- link summit_xls_front_right_wheel_link: geometry collision cylinder length=0.087 radius=0.127; visual mesh filename=/home/ubuntu/Rofunc/rofunc/simulator/assets/urdf/curi_descr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
- link torso_base1: geometry collision mesh filename=/home/ubuntu/Rofunc/rofunc/simulator/assets/urdf/curi_descr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; visual mesh filename=/home/ubuntu/Rofunc/rofunc/simulator/assets/urdf/curi_descr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
- link torso_base2: geometry collision mesh filename=/home/ubuntu/Rofunc/rofunc/simulator/assets/urdf/curi_descr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; visual mesh filename=/home/ubuntu/Rofunc/rofunc/simulator/assets/urdf/curi_descr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
- link torso_end: geometry collision mesh filename=/home/ubuntu/Rofunc/rofunc/simulator/assets/urdf/curi_descr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; visual mesh filename=/home/ubuntu/Rofunc/rofunc/simulator/assets/urdf/curi_descr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
- link torso_link_b1: geometry collision mesh filename=/home/ubuntu/Rofunc/rofunc/simulator/assets/urdf/curi_descr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; visual mesh filename=/home/ubuntu/Rofunc/rofunc/simulator/assets/urdf/curi_descr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
- link torso_link_b2: geometry collision mesh filename=/home/ubuntu/Rofunc/rofunc/simulator/assets/urdf/curi_descr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; visual mesh filename=/home/ubuntu/Rofunc/rofunc/simulator/assets/urdf/curi_descr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
- link torso_link_c1: geometry collision mesh filename=/home/ubuntu/Rofunc/rofunc/simulator/assets/urdf/curi_descr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; visual mesh filename=/home/ubuntu/Rofunc/rofunc/simulator/assets/urdf/curi_descr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
- link torso_link_c2: geometry collision mesh filename=/home/ubuntu/Rofunc/rofunc/simulator/assets/urdf/curi_descr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; visual mesh filename=/home/ubuntu/Rofunc/rofunc/simulator/assets/urdf/curi_descr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
- link torso_middle: geometry collision mesh filename=/home/ubuntu/Rofunc/rofunc/simulator/assets/urdf/curi_descr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; visual mesh filename=/home/ubuntu/Rofunc/rofunc/simulator/assets/urdf/curi_descr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

File: rofunc/simulator/assets/urdf/curi/urdf/robotnik/summit_xls.urdf (robot description, URDF)
Before this commit: robot summit_xls, 7 links, 6 joints
Links:
- link summit_xls_back_left_wheel_link: geometry collision cylinder length=0.087 radius=0.127; visual mesh filename=/home/ubuntu/Rofunc/rofunc/simulator/assets/urdf/curi_descr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
- link summit_xls_back_right_wheel_link: geometry collision cylinder length=0.087 radius=0.127; visual mesh filename=/home/ubuntu/Rofunc/rofunc/simulator/assets/urdf/curi_descr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
- link summit_xls_base_link: geometry collision mesh filename=/home/ubuntu/Rofunc/rofunc/simulator/assets/urdf/curi_descr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; visual mesh filename=/home/ubuntu/Rofunc/rofunc/simulator/assets/urdf/curi_descr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
- link summit_xls_front_left_wheel_link: geometry collision cylinder length=0.087 radius=0.127; visual mesh filename=/home/ubuntu/Rofunc/rofunc/simulator/assets/urdf/curi_descr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
- link summit_xls_front_right_wheel_link: geometry collision cylinder length=0.087 radius=0.127; visual mesh filename=/home/ubuntu/Rofunc/rofunc/simulator/assets/urdf/curi_descr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

File: rofunc/simulator/assets/urdf/curi/urdf/robotnik/summit_xls_gazebo.urdf (robot description, URDF)
Before this commit: robot summit_xls, 6 links, 5 joints
Links:
- link summit_xls_back_left_wheel_link: geometry collision cylinder length=0.087 radius=0.127; visual mesh filename=/home/ubuntu/Rofunc/rofunc/simulator/assets/urdf/curi_descr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
- link summit_xls_back_right_wheel_link: geometry collision cylinder length=0.087 radius=0.127; visual mesh filename=/home/ubuntu/Rofunc/rofunc/simulator/assets/urdf/curi_descr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
- link summit_xls_base_link: geometry collision mesh filename=/home/ubuntu/Rofunc/rofunc/simulator/assets/urdf/curi_descr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; visual mesh filename=/home/ubuntu/Rofunc/rofunc/simulator/assets/urdf/curi_descr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
- link summit_xls_front_left_wheel_link: geometry collision cylinder length=0.087 radius=0.127; visual mesh filename=/home/ubuntu/Rofunc/rofunc/simulator/assets/urdf/curi_descr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
- link summit_xls_front_right_wheel_link: geometry collision cylinder length=0.087 radius=0.127; visual mesh filename=/home/ubuntu/Rofunc/rofunc/simulator/assets/urdf/curi_descr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

File: rofunc/simulator/assets/urdf/franka_description/robots/franka_panda.urdf (robot description, URDF)
Before this commit: robot panda, 11 links, 10 joints
Links:
- link panda_hand: geometry collision mesh filename=/home/ubuntu/Rofunc/rofunc/simulator/assets/urdf/franka_des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; visual mesh filename=/home/ubuntu/Rofunc/rofunc/simulator/assets/urdf/franka_des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
- link panda_leftfinger: geometry collision mesh filename=/home/ubuntu/Rofunc/rofunc/simulator/assets/urdf/franka_des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; visual mesh filename=/home/ubuntu/Rofunc/rofunc/simulator/assets/urdf/franka_des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
- link panda_link0: geometry collision mesh filename=/home/ubuntu/Rofunc/rofunc/simulator/assets/urdf/franka_des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; visual mesh filename=/home/ubuntu/Rofunc/rofunc/simulator/assets/urdf/franka_des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
- link panda_link1: geometry collision mesh filename=/home/ubuntu/Rofunc/rofunc/simulator/assets/urdf/franka_des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; visual mesh filename=/home/ubuntu/Rofunc/rofunc/simulator/assets/urdf/franka_des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
- link panda_link2: geometry collision mesh filename=/home/ubuntu/Rofunc/rofunc/simulator/assets/urdf/franka_des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; visual mesh filename=/home/ubuntu/Rofunc/rofunc/simulator/assets/urdf/franka_des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
- link panda_link3: geometry collision mesh filename=/home/ubuntu/Rofunc/rofunc/simulator/assets/urdf/franka_des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; visual mesh filename=/home/ubuntu/Rofunc/rofunc/simulator/assets/urdf/franka_des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
- link panda_link4: geometry collision mesh filename=/home/ubuntu/Rofunc/rofunc/simulator/assets/urdf/franka_des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; visual mesh filename=/home/ubuntu/Rofunc/rofunc/simulator/assets/urdf/franka_des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
- link panda_link5: geometry collision mesh filename=/home/ubuntu/Rofunc/rofunc/simulator/assets/urdf/franka_des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; visual mesh filename=/home/ubuntu/Rofunc/rofunc/simulator/assets/urdf/franka_des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
- link panda_link6: geometry collision mesh filename=/home/ubuntu/Rofunc/rofunc/simulator/assets/urdf/franka_des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; visual mesh filename=/home/ubuntu/Rofunc/rofunc/simulator/assets/urdf/franka_des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
- link panda_link7: geometry collision mesh filename=/home/ubuntu/Rofunc/rofunc/simulator/assets/urdf/franka_des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; visual mesh filename=/home/ubuntu/Rofunc/rofunc/simulator/assets/urdf/franka_des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
- link panda_rightfinger: geometry collision mesh filename=/home/ubuntu/Rofunc/rofunc/simulator/assets/urdf/franka_des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; visual mesh filename=/home/ubuntu/Rofunc/rofunc/simulator/assets/urdf/franka_des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
