Commit message: update urdf

File: rofunc/simulator/assets/urdf/kinova_description/urdf/kinova.urdf (robot description, URDF)
Before this commit: robot kinova, 14 links, 13 joints
Links:
- link kinova_link_1: geometry collision mesh filename=/home/ubuntu/Rofunc/rofunc/simulator/assets/urdf/kinova_des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; visual mesh filename=/home/ubuntu/Rofunc/rofunc/simulator/assets/urdf/kinova_des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
- link kinova_link_2: geometry collision mesh filename=/home/ubuntu/Rofunc/rofunc/simulator/assets/urdf/kinova_des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; visual mesh filename=/home/ubuntu/Rofunc/rofunc/simulator/assets/urdf/kinova_des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
- link kinova_link_3: geometry collision mesh filename=/home/ubuntu/Rofunc/rofunc/simulator/assets/urdf/kinova_des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; visual mesh filename=/home/ubuntu/Rofunc/rofunc/simulator/assets/urdf/kinova_des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
- link kinova_link_4: geometry collision mesh filename=/home/ubuntu/Rofunc/rofunc/simulator/assets/urdf/kinova_des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; visual mesh filename=/home/ubuntu/Rofunc/rofunc/simulator/assets/urdf/kinova_des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
- link kinova_link_5: geometry collision mesh filename=/home/ubuntu/Rofunc/rofunc/simulator/assets/urdf/kinova_des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; visual mesh filename=/home/ubuntu/Rofunc/rofunc/simulator/assets/urdf/kinova_des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
- link kinova_link_6: geometry collision mesh filename=/home/ubuntu/Rofunc/rofunc/simulator/assets/urdf/kinova_des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; visual mesh filename=/home/ubuntu/Rofunc/rofunc/simulator/assets/urdf/kinova_des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
- link kinova_link_base: geometry collision mesh filename=/home/ubuntu/Rofunc/rofunc/simulator/assets/urdf/kinova_des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; visual mesh filename=/home/ubuntu/Rofunc/rofunc/simulator/assets/urdf/kinova_des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
- link kinova_link_finger_1: geometry collision mesh filename=/home/ubuntu/Rofunc/rofunc/simulator/assets/urdf/kinova_des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; visual mesh filename=/home/ubuntu/Rofunc/rofunc/simulator/assets/urdf/kinova_des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
- link kinova_link_finger_2: geometry collision mesh filename=/home/ubuntu/Rofunc/rofunc/simulator/assets/urdf/kinova_des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; visual mesh filename=/home/ubuntu/Rofunc/rofunc/simulator/assets/urdf/kinova_des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
- link kinova_link_finger_3: geometry collision mesh filename=/home/ubuntu/Rofunc/rofunc/simulator/assets/urdf/kinova_des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; visual mesh filename=/home/ubuntu/Rofunc/rofunc/simulator/assets/urdf/kinova_des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
- link kinova_link_finger_tip_1: geometry collision mesh filename=/home/ubuntu/Rofunc/rofunc/simulator/assets/urdf/kinova_des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; visual mesh filename=/home/ubuntu/Rofunc/rofunc/simulator/assets/urdf/kinova_des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
- link kinova_link_finger_tip_2: geometry collision mesh filename=/home/ubuntu/Rofunc/rofunc/simulator/assets/urdf/kinova_des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; visual mesh filename=/home/ubuntu/Rofunc/rofunc/simulator/assets/urdf/kinova_des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
- link kinova_link_finger_tip_3: geometry collision mesh filename=/home/ubuntu/Rofunc/rofunc/simulator/assets/urdf/kinova_des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; visual mesh filename=/home/ubuntu/Rofunc/rofunc/simulator/assets/urdf/kinova_des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
