Commit message: format update

File: rofunc/simulator/assets/urdf/curi/urdf/curi_cartesio.urdf (robot description, URDF)
Before this commit: robot curi, 35 links, 34 joints
Links:
- link control_box: geometry collision mesh filename=../meshes/clover/collision/control_box.stl; visual mesh filename=../meshes/clover/visual/control_box.dae
- link head_base: geometry collision mesh filename=../meshes/clover/collision/head_base.stl; visual mesh filename=../meshes/clover/visual/head_base.dae
- link head_link1: geometry collision mesh filename=../meshes/clover/collision/head_link1.stl; visual mesh filename=../meshes/clover/visual/head_link1.dae
- link head_link2: geometry collision mesh filename=../meshes/clover/collision/head_link2.stl; visual mesh filename=../meshes/clover/visual/head_link2.dae
- link panda_left_hand: geometry collision mesh filename=../meshes/franka/collision/hand.stl; visual mesh filename=../meshes/franka/visual/hand.dae
- link panda_left_link0: geometry collision mesh filename=../meshes/franka/collision/link0.stl; visual mesh filename=../meshes/franka/visual/link0.dae
- link panda_left_link1: geometry collision mesh filename=../meshes/franka/collision/link1.stl; visual mesh filename=../meshes/franka/visual/link1.dae
- link panda_left_link2: geometry collision mesh filename=../meshes/franka/collision/link2.stl; visual mesh filename=../meshes/franka/visual/link2.dae
- link panda_left_link3: geometry collision mesh filename=../meshes/franka/collision/link3.stl; visual mesh filename=../meshes/franka/visual/link3.dae
- link panda_left_link4: geometry collision mesh filename=../meshes/franka/collision/link4.stl; visual mesh filename=../meshes/franka/visual/link4.dae
- link panda_left_link5: geometry collision mesh filename=../meshes/franka/collision/link5.stl; visual mesh filename=../meshes/franka/visual/link5.dae
- link panda_left_link6: geometry collision mesh filename=../meshes/franka/collision/link6.stl; visual mesh filename=../meshes/franka/visual/link6.dae
- link panda_left_link7: geometry collision mesh filename=../meshes/franka/collision/link7.stl; visual mesh filename=../meshes/franka/visual/link7.dae
- link panda_right_hand: geometry collision mesh filename=../meshes/franka/collision/hand.stl; visual mesh filename=../meshes/franka/visual/hand.dae
- link panda_right_link0: geometry collision mesh filename=../meshes/franka/collision/link0.stl; visual mesh filename=../meshes/franka/visual/link0.dae
- link panda_right_link1: geometry collision mesh filename=../meshes/franka/collision/link1.stl; visual mesh filename=../meshes/franka/visual/link1.dae
- link panda_right_link2: geometry collision mesh filename=../meshes/franka/collision/link2.stl; visual mesh filename=../meshes/franka/visual/link2.dae
- link panda_right_link3: geometry collision mesh filename=../meshes/franka/collision/link3.stl; visual mesh filename=../meshes/franka/visual/link3.dae
- link panda_right_link4: geometry collision mesh filename=../meshes/franka/collision/link4.stl; visual mesh filename=../meshes/franka/visual/link4.dae
- link panda_right_link5: geometry collision mesh filename=../meshes/franka/collision/link5.stl; visual mesh filename=../meshes/franka/visual/link5.dae
- link panda_right_link6: geometry collision mesh filename=../meshes/franka/collision/link6.stl; visual mesh filename=../meshes/franka/visual/link6.dae
- link panda_right_link7: geometry collision mesh filename=../meshes/franka/collision/link7.stl; visual mesh filename=../meshes/franka/visual/link7.dae
- link summit_xls_back_left_wheel_link: geometry collision cylinder length=0.087 radius=0.127; visual mesh filename=../meshes/robotnik/wheels/omni_wheel_1.dae
- link summit_xls_back_right_wheel_link: geometry collision cylinder length=0.087 radius=0.127; visual mesh filename=../meshes/robotnik/wheels/omni_wheel_2.dae
- link summit_xls_base_link: geometry collision mesh filename=../meshes/robotnik/bases/summit_xls_chassis.stl; visual mesh filename=../meshes/robotnik/bases/summit_xls_chassis.dae
- link summit_xls_front_left_wheel_link: geometry collision cylinder length=0.087 radius=0.127; visual mesh filename=../meshes/robotnik/wheels/omni_wheel_1.dae
- link summit_xls_front_right_wheel_link: geometry collision cylinder length=0.087 radius=0.127; visual mesh filename=../meshes/robotnik/wheels/omni_wheel_2.dae
- link torso_base1: geometry collision mesh filename=../meshes/clover/collision/torso_base1.stl; visual mesh filename=../meshes/clover/visual/torso_base1.dae
- link torso_base2: geometry collision mesh filename=../meshes/clover/collision/torso_base2.stl; visual mesh filename=../meshes/clover/visual/torso_base2.dae
- link torso_end: geometry collision mesh filename=../meshes/clover/collision/torso_end.stl; visual mesh filename=../meshes/clover/visual/torso_end.dae
- link torso_link_b2: geometry collision mesh filename=../meshes/clover/collision/torso_link_b2.stl; visual mesh filename=../meshes/clover/visual/torso_link_b2.dae
- link torso_link_c1: geometry collision mesh filename=../meshes/clover/collision/torso_link_c1.stl; visual mesh filename=../meshes/clover/visual/torso_link_c1.dae
- link torso_middle: geometry collision mesh filename=../meshes/clover/collision/torso_middle.stl; visual mesh filename=../meshes/clover/visual/torso_middle.dae

File: rofunc/simulator/assets/urdf/curi/urdf/curi_mujoco.urdf (robot description, URDF)
Before this commit: robot curi, 41 links, 40 joints
Links:
- link control_box: geometry collision mesh filename=../meshes/clover/collision/control_box.stl; visual mesh filename=../meshes/clover/visual/control_box.dae
- link head_base: geometry collision mesh filename=../meshes/clover/collision/head_base.stl; visual mesh filename=../meshes/clover/visual/head_base.dae
- link head_link1: geometry collision mesh filename=../meshes/clover/collision/head_link1.stl; visual mesh filename=../meshes/clover/visual/head_link1.dae
- link head_link2: geometry collision mesh filename=../meshes/clover/collision/head_link2.stl; visual mesh filename=../meshes/clover/visual/head_link2.dae
- link panda_left_hand: geometry collision mesh filename=../meshes/franka/collision/hand.stl; visual mesh filename=../meshes/franka/visual/hand.dae
- link panda_left_leftfinger: geometry collision box size=17.5e-3 15.2e-3 18.5e-3; collision box size=17.5e-3 7e-3 23.5e-3
- link panda_left_link0: geometry collision mesh filename=../meshes/franka/collision/link0.stl; visual mesh filename=../meshes/franka/visual/link0.dae
- link panda_left_link1: geometry collision mesh filename=../meshes/franka/collision/link1.stl; visual mesh filename=../meshes/franka/visual/link1.dae
- link panda_left_link2: geometry collision mesh filename=../meshes/franka/collision/link2.stl; visual mesh filename=../meshes/franka/visual/link2.dae
- link panda_left_link3: geometry collision mesh filename=../meshes/franka/collision/link3.stl; visual mesh filename=../meshes/franka/visual/link3.dae
- link panda_left_link4: geometry collision mesh filename=../meshes/franka/collision/link4.stl; visual mesh filename=../meshes/franka/visual/link4.dae
- link panda_left_link5: geometry collision mesh filename=../meshes/franka/collision/link5.stl; visual mesh filename=../meshes/franka/visual/link5.dae
- link panda_left_link6: geometry collision mesh filename=../meshes/franka/collision/link6.stl; visual mesh filename=../meshes/franka/visual/link6.dae
- link panda_left_link7: geometry collision mesh filename=../meshes/franka/collision/link7.stl; visual mesh filename=../meshes/franka/visual/link7.dae
- link panda_left_rightfinger: geometry collision box size=17.5e-3 15.2e-3 18.5e-3; collision box size=17.5e-3 7e-3 23.5e-3
- link panda_right_hand: geometry collision mesh filename=../meshes/franka/collision/hand.stl; visual mesh filename=../meshes/franka/visual/hand.dae
- link panda_right_leftfinger: geometry collision box size=17.5e-3 15.2e-3 18.5e-3; collision box size=17.5e-3 7e-3 23.5e-3
- link panda_right_link0: geometry collision mesh filename=../meshes/franka/collision/link0.stl; visual mesh filename=../meshes/franka/visual/link0.dae
- link panda_right_link1: geometry collision mesh filename=../meshes/franka/collision/link1.stl; visual mesh filename=../meshes/franka/visual/link1.dae
- link panda_right_link2: geometry collision mesh filename=../meshes/franka/collision/link2.stl; visual mesh filename=../meshes/franka/visual/link2.dae
- link panda_right_link3: geometry collision mesh filename=../meshes/franka/collision/link3.stl; visual mesh filename=../meshes/franka/visual/link3.dae
- link panda_right_link4: geometry collision mesh filename=../meshes/franka/collision/link4.stl; visual mesh filename=../meshes/franka/visual/link4.dae
- link panda_right_link5: geometry collision mesh filename=../meshes/franka/collision/link5.stl; visual mesh filename=../meshes/franka/visual/link5.dae
- link panda_right_link6: geometry collision mesh filename=../meshes/franka/collision/link6.stl; visual mesh filename=../meshes/franka/visual/link6.dae
- link panda_right_link7: geometry collision mesh filename=../meshes/franka/collision/link7.stl; visual mesh filename=../meshes/franka/visual/link7.dae
- link panda_right_rightfinger: geometry collision box size=17.5e-3 15.2e-3 18.5e-3; collision box size=17.5e-3 7e-3 23.5e-3
- link summit_xls_back_left_wheel_link: geometry collision cylinder length=0.087 radius=0.127; visual mesh filename=../meshes/robotnik/wheels/omni_wheel_1.dae
- link summit_xls_back_right_wheel_link: geometry collision cylinder length=0.087 radius=0.127; visual mesh filename=../meshes/robotnik/wheels/omni_wheel_2.dae
- link summit_xls_base_link: geometry collision mesh filename=../meshes/robotnik/bases/summit_xls_chassis.stl; visual mesh filename=../meshes/robotnik/bases/summit_xls_chassis.dae
- link summit_xls_front_left_wheel_link: geometry collision cylinder length=0.087 radius=0.127; visual mesh filename=../meshes/robotnik/wheels/omni_wheel_1.dae
- link summit_xls_front_right_wheel_link: geometry collision cylinder length=0.087 radius=0.127; visual mesh filename=../meshes/robotnik/wheels/omni_wheel_2.dae
- link torso_base1: geometry collision mesh filename=../meshes/clover/collision/torso_base1.stl; visual mesh filename=../meshes/clover/visual/torso_base1.dae
- link torso_base2: geometry collision mesh filename=../meshes/clover/collision/torso_base2.stl; visual mesh filename=../meshes/clover/visual/torso_base2.dae
- link torso_end: geometry collision mesh filename=../meshes/clover/collision/torso_end.stl; visual mesh filename=../meshes/clover/visual/torso_end.dae
- link torso_link_b1: geometry collision mesh filename=../meshes/clover/collision/torso_link_b1.stl; visual mesh filename=../meshes/clover/visual/torso_link_b1.dae
- link torso_link_b2: geometry collision mesh filename=../meshes/clover/collision/torso_link_b2.stl; visual mesh filename=../meshes/clover/visual/torso_link_b2.dae
- link torso_link_c1: geometry collision mesh filename=../meshes/clover/collision/torso_link_c1.stl; visual mesh filename=../meshes/clover/visual/torso_link_c1.dae
- link torso_link_c2: geometry collision mesh filename=../meshes/clover/collision/torso_link_c2.stl; visual mesh filename=../meshes/clover/visual/torso_link_c2.dae
- link torso_middle: geometry collision mesh filename=../meshes/clover/collision/torso_middle.stl; visual mesh filename=../meshes/clover/visual/torso_middle.dae

File: rofunc/simulator/assets/urdf/curi/urdf/robotnik/summit_xls.urdf (robot description, URDF)
Before this commit: robot summit_xls, 7 links, 6 joints
Links:
- link summit_xls_back_left_wheel_link: geometry collision cylinder length=0.087 radius=0.127; visual mesh filename=../meshes/robotnik/wheels/omni_wheel_1.dae
- link summit_xls_back_right_wheel_link: geometry collision cylinder length=0.087 radius=0.127; visual mesh filename=../meshes/robotnik/wheels/omni_wheel_2.dae
- link summit_xls_base_link: geometry collision mesh filename=../meshes/robotnik/bases/summit_xls_chassis.stl; visual mesh filename=../meshes/robotnik/bases/summit_xls_chassis.dae
- link summit_xls_front_left_wheel_link: geometry collision cylinder length=0.087 radius=0.127; visual mesh filename=../meshes/robotnik/wheels/omni_wheel_1.dae
- link summit_xls_front_right_wheel_link: geometry collision cylinder length=0.087 radius=0.127; visual mesh filename=../meshes/robotnik/wheels/omni_wheel_2.dae

File: rofunc/simulator/assets/urdf/curi/urdf/robotnik/summit_xls_gazebo.urdf (robot description, URDF)
Before this commit: robot summit_xls, 6 links, 5 joints
Links:
- link summit_xls_back_left_wheel_link: geometry collision cylinder length=0.087 radius=0.127; visual mesh filename=../meshes/robotnik/wheels/omni_wheel_1.dae
- link summit_xls_back_right_wheel_link: geometry collision cylinder length=0.087 radius=0.127; visual mesh filename=../meshes/robotnik/wheels/omni_wheel_2.dae
- link summit_xls_base_link: geometry collision mesh filename=../meshes/robotnik/bases/summit_xls_chassis.stl; visual mesh filename=../meshes/robotnik/bases/summit_xls_chassis.dae
- link summit_xls_front_left_wheel_link: geometry collision cylinder length=0.087 radius=0.127; visual mesh filename=../meshes/robotnik/wheels/omni_wheel_1.dae
- link summit_xls_front_right_wheel_link: geometry collision cylinder length=0.087 radius=0.127; visual mesh filename=../meshes/robotnik/wheels/omni_wheel_2.dae
