Commit message: Update the newest CURI model and add yup urdf file for Isaac Gym

File: rofunc/simulator/assets/urdf/curi/urdf/curi_isaacgym.urdf (robot description, URDF)
Before this commit: robot curi, 39 links, 38 joints
Links:
- link torso_end: geometry collision mesh filename=../meshes/clover/collision/torso_end_v2_yup.stl; visual mesh filename=../meshes/clover/visual/torso_end_v2_yup.dae
Joints:
- joint head_joint_torso_end: origin xyz=0.01466 0 0.2775 rpy=0 0 0 -> xyz=0.02 0 0.3929 rpy=0 0 0
- joint panda_left_joint_torso_end: origin xyz=0.02842 0.11216 0.19004 rpy=-1.5004311592913677 0.8772798703277918 -0.2038499389018784 -> xyz=-0.08537 0.07009 0.2535 rpy=-1.3685238493647454 0.913218224774749 -0.6168337646727412
- joint panda_right_joint_torso_end: origin xyz=0.02842 -0.11216 0.19004 rpy=1.5004311592913677 0.8772798703277918 0.2038499389018784 -> xyz=-0.08537 -0.07009 0.2535 rpy=1.3685238493647454 0.913218224774749 0.6168337646727412

File: rofunc/simulator/assets/urdf/curi/urdf/curi_w_softhand_isaacgym.urdf (robot description, URDF)
Before this commit: robot curi, 111 links, 110 joints
Links:
- removed link torso_link_b1
- removed link torso_link_c2
- link left_qbhand_base_link: geometry collision mesh filename=../meshes/qbhand/flange_iso_04_yupzfront.STL scale=1 1 1; visual mesh filename=../meshes/qbhand/flange_iso_04_yupzfront.STL scale=1 1 1
- link left_qbhand_index_distal_link: geometry collision mesh filename=../meshes/qbhand/ph_distal_yupzfront1.STL scale=1 1 1; visual mesh filename=../meshes/qbhand/ph_distal_yupzfront1.STL scale=1 1 1
- link left_qbhand_index_knuckle_link: geometry collision mesh filename=../meshes/qbhand/ph_knuckle_yupzfront1.STL scale=1 1 1; visual mesh filename=../meshes/qbhand/ph_knuckle_yupzfront1.STL scale=1 1 1
- link left_qbhand_index_middle_link: geometry collision mesh filename=../meshes/qbhand/ph_short_yupzfront1.STL scale=1 1 1; visual mesh filename=../meshes/qbhand/ph_short_yupzfront1.STL scale=1 1 1
- link left_qbhand_index_proximal_link: geometry collision mesh filename=../meshes/qbhand/ph_medium_yupzfront1.STL scale=1 1 1; visual mesh filename=../meshes/qbhand/ph_medium_yupzfront1.STL scale=1 1 1
- link left_qbhand_little_distal_link: geometry collision mesh filename=../meshes/qbhand/ph_distal_yupzfront1.STL scale=1 1 1; visual mesh filename=../meshes/qbhand/ph_distal_yupzfront1.STL scale=1 1 1
- link left_qbhand_little_knuckle_link: geometry collision mesh filename=../meshes/qbhand/ph_knuckle_yupzfront1.STL scale=1 1 1; visual mesh filename=../meshes/qbhand/ph_knuckle_yupzfront1.STL scale=1 1 1
- link left_qbhand_little_middle_link: geometry collision mesh filename=../meshes/qbhand/ph_short_yupzfront1.STL scale=1 1 1; visual mesh filename=../meshes/qbhand/ph_short_yupzfront1.STL scale=1 1 1
- link left_qbhand_little_proximal_link: geometry collision mesh filename=../meshes/qbhand/ph_short_yupzfront1.STL scale=1 1 1; visual mesh filename=../meshes/qbhand/ph_short_yupzfront1.STL scale=1 1 1
- link left_qbhand_middle_distal_link: geometry collision mesh filename=../meshes/qbhand/ph_distal_yupzfront1.STL scale=1 1 1; visual mesh filename=../meshes/qbhand/ph_distal_yupzfront1.STL scale=1 1 1
- link left_qbhand_middle_knuckle_link: geometry collision mesh filename=../meshes/qbhand/ph_knuckle_yupzfront1.STL scale=1 1 1; visual mesh filename=../meshes/qbhand/ph_knuckle_yupzfront1.STL scale=1 1 1
- link left_qbhand_middle_middle_link: geometry collision mesh filename=../meshes/qbhand/ph_short_yupzfront1.STL scale=1 1 1; visual mesh filename=../meshes/qbhand/ph_short_yupzfront1.STL scale=1 1 1
- link left_qbhand_middle_proximal_link: geometry collision mesh filename=../meshes/qbhand/ph_medium_yupzfront1.STL scale=1 1 1; visual mesh filename=../meshes/qbhand/ph_medium_yupzfront1.STL scale=1 1 1
- link left_qbhand_palm_link: geometry collision mesh filename=../meshes/qbhand/palm_pinch_l_yupzfront1.STL scale=1000 1000 1000; visual mesh filename=../meshes/qbhand/palm_pinch_l_yupzfront1.STL scale=1000 1000 1000
- link left_qbhand_ring_distal_link: geometry collision mesh filename=../meshes/qbhand/ph_distal_yupzfront1.STL scale=1 1 1; visual mesh filename=../meshes/qbhand/ph_distal_yupzfront1.STL scale=1 1 1
- link left_qbhand_ring_knuckle_link: geometry collision mesh filename=../meshes/qbhand/ph_knuckle_yupzfront1.STL scale=1 1 1; visual mesh filename=../meshes/qbhand/ph_knuckle_yupzfront1.STL scale=1 1 1
- link left_qbhand_ring_middle_link: geometry collision mesh filename=../meshes/qbhand/ph_short_yupzfront1.STL scale=1 1 1; visual mesh filename=../meshes/qbhand/ph_short_yupzfront1.STL scale=1 1 1
- link left_qbhand_ring_proximal_link: geometry collision mesh filename=../meshes/qbhand/ph_medium_yupzfront1.STL scale=1 1 1; visual mesh filename=../meshes/qbhand/ph_medium_yupzfront1.STL scale=1 1 1
- link left_qbhand_thumb_distal_link: geometry collision mesh filename=../meshes/qbhand/ph_distal_yupzfront1.STL scale=1 1 1; visual mesh filename=../meshes/qbhand/ph_distal_yupzfront1.STL scale=1 1 1
- link left_qbhand_thumb_knuckle_link: geometry collision mesh filename=../meshes/qbhand/ph_thumb_l_yupzfront1.STL scale=1 1 1; visual mesh filename=../meshes/qbhand/ph_thumb_l_yupzfront1.STL scale=1 1 1
- link left_qbhand_thumb_proximal_link: geometry collision mesh filename=../meshes/qbhand/ph_short_yupzfront1.STL scale=1 1 1; visual mesh filename=../meshes/qbhand/ph_short_yupzfront1.STL scale=1 1 1
- link right_qbhand_base_link: geometry collision mesh filename=../meshes/qbhand/flange_iso_04_yupzfront.STL scale=1 1 1; visual mesh filename=../meshes/qbhand/flange_iso_04_yupzfront.STL scale=1 1 1
- link right_qbhand_index_distal_link: geometry collision mesh filename=../meshes/qbhand/ph_distal_yupzfront1.STL scale=1 1 1; visual mesh filename=../meshes/qbhand/ph_distal_yupzfront1.STL scale=1 1 1
- link right_qbhand_index_knuckle_link: geometry collision mesh filename=../meshes/qbhand/ph_knuckle_yupzfront1.STL scale=1 1 1; visual mesh filename=../meshes/qbhand/ph_knuckle_yupzfront1.STL scale=1 1 1
- link right_qbhand_index_middle_link: geometry collision mesh filename=../meshes/qbhand/ph_short_yupzfront1.STL scale=1 1 1; visual mesh filename=../meshes/qbhand/ph_short_yupzfront1.STL scale=1 1 1
- link right_qbhand_index_proximal_link: geometry collision mesh filename=../meshes/qbhand/ph_medium_yupzfront1.STL scale=1 1 1; visual mesh filename=../meshes/qbhand/ph_medium_yupzfront1.STL scale=1 1 1
- link right_qbhand_little_distal_link: geometry collision mesh filename=../meshes/qbhand/ph_distal_yupzfront1.STL scale=1 1 1; visual mesh filename=../meshes/qbhand/ph_distal_yupzfront1.STL scale=1 1 1
- link right_qbhand_little_knuckle_link: geometry collision mesh filename=../meshes/qbhand/ph_knuckle_yupzfront1.STL scale=1 1 1; visual mesh filename=../meshes/qbhand/ph_knuckle_yupzfront1.STL scale=1 1 1
- link right_qbhand_little_middle_link: geometry collision mesh filename=../meshes/qbhand/ph_short_yupzfront1.STL scale=1 1 1; visual mesh filename=../meshes/qbhand/ph_short_yupzfront1.STL scale=1 1 1
- link right_qbhand_little_proximal_link: geometry collision mesh filename=../meshes/qbhand/ph_short_yupzfront1.STL scale=1 1 1; visual mesh filename=../meshes/qbhand/ph_short_yupzfront1.STL scale=1 1 1
- link right_qbhand_middle_distal_link: geometry collision mesh filename=../meshes/qbhand/ph_distal_yupzfront1.STL scale=1 1 1; visual mesh filename=../meshes/qbhand/ph_distal_yupzfront1.STL scale=1 1 1
- link right_qbhand_middle_knuckle_link: geometry collision mesh filename=../meshes/qbhand/ph_knuckle_yupzfront1.STL scale=1 1 1; visual mesh filename=../meshes/qbhand/ph_knuckle_yupzfront1.STL scale=1 1 1
- link right_qbhand_middle_middle_link: geometry collision mesh filename=../meshes/qbhand/ph_short_yupzfront1.STL scale=1 1 1; visual mesh filename=../meshes/qbhand/ph_short_yupzfront1.STL scale=1 1 1
- link right_qbhand_middle_proximal_link: geometry collision mesh filename=../meshes/qbhand/ph_medium_yupzfront1.STL scale=1 1 1; visual mesh filename=../meshes/qbhand/ph_medium_yupzfront1.STL scale=1 1 1
- link right_qbhand_palm_link: geometry collision mesh filename=../meshes/qbhand/palm_pinch_r.stl scale=0.001 0.001 0.001; visual mesh filename=../meshes/qbhand/palm_pinch_r_yupzfront2.STL scale=1 1 1
- link right_qbhand_ring_distal_link: geometry collision mesh filename=../meshes/qbhand/ph_distal_yupzfront1.STL scale=1 1 1; visual mesh filename=../meshes/qbhand/ph_distal_yupzfront1.STL scale=1 1 1
- link right_qbhand_ring_knuckle_link: geometry collision mesh filename=../meshes/qbhand/ph_knuckle_yupzfront1.STL scale=1 1 1; visual mesh filename=../meshes/qbhand/ph_knuckle_yupzfront1.STL scale=1 1 1
- link right_qbhand_ring_middle_link: geometry collision mesh filename=../meshes/qbhand/ph_short_yupzfront1.STL scale=1 1 1; visual mesh filename=../meshes/qbhand/ph_short_yupzfront1.STL scale=1 1 1
- link right_qbhand_ring_proximal_link: geometry collision mesh filename=../meshes/qbhand/ph_medium_yupzfront1.STL scale=1 1 1; visual mesh filename=../meshes/qbhand/ph_medium_yupzfront1.STL scale=1 1 1
- link right_qbhand_thumb_distal_link: geometry collision mesh filename=../meshes/qbhand/ph_distal_yupzfront1.STL scale=1 1 1; visual mesh filename=../meshes/qbhand/ph_distal_yupzfront1.STL scale=1 1 1
- link right_qbhand_thumb_knuckle_link: geometry collision mesh filename=../meshes/qbhand/ph_thumb_r_yupzfront1.STL scale=1 1 1; visual mesh filename=../meshes/qbhand/ph_thumb_r_yupzfront1.STL scale=1 1 1
- link right_qbhand_thumb_proximal_link: geometry collision mesh filename=../meshes/qbhand/ph_short_yupzfront1.STL scale=1 1 1; visual mesh filename=../meshes/qbhand/ph_short_yupzfront1.STL scale=1 1 1
- link torso_end: geometry collision mesh filename=../meshes/clover/collision/torso_end_v2_yup.stl; visual mesh filename=../meshes/clover/visual/torso_end_v2_yup.dae
Joints:
- removed joint torso_joint4
- removed joint torso_joint7
- joint left_qbhand_thumb_knuckle_joint: axis 0 0 -1 -> 0 0 1
- joint torso_actuated_joint2: axis 0 1 0 -> (none); limit lower=-1.2 upper=0.5 effort=300 velocity=0.3 -> (none); type revolute -> fixed
- joint torso_actuated_joint3: axis 0 1 0 -> (none); limit lower=-0.9 upper=0.9 effort=300 velocity=0.3 -> (none); type revolute -> fixed
- joint torso_joint5: axis 0 1 0 -> (none); limit lower=-0.5 upper=1.2 effort=300 velocity=0.3 -> (none); mimic joint=torso_actuated_joint2 multiplier=-1 -> (none); type revolute -> fixed
- joint torso_joint8: axis 0 1 0 -> (none); limit lower=-0.9 upper=0.9 effort=300 velocity=0.3 -> (none); mimic joint=torso_actuated_joint3 multiplier=-1 -> (none); type revolute -> fixed

File: rofunc/simulator/assets/urdf/curi/urdf/curi_w_softhand_yup.urdf (robot description, URDF)
Before this commit: robot curi, 111 links, 110 joints
Links:
- link left_qbhand_base_link: geometry collision mesh filename=../meshes/qbhand/flange_iso_04_yupzfront.STL scale=1 1 1; visual mesh filename=../meshes/qbhand/flange_iso_04_yupzfront.STL scale=1 1 1
- link left_qbhand_index_distal_link: geometry collision mesh filename=../meshes/qbhand/ph_distal_yupzfront1.STL scale=1 1 1; visual mesh filename=../meshes/qbhand/ph_distal_yupzfront1.STL scale=1 1 1
- link left_qbhand_index_knuckle_link: geometry collision mesh filename=../meshes/qbhand/ph_knuckle_yupzfront1.STL scale=1 1 1; visual mesh filename=../meshes/qbhand/ph_knuckle_yupzfront1.STL scale=1 1 1
- link left_qbhand_index_middle_link: geometry collision mesh filename=../meshes/qbhand/ph_short_yupzfront1.STL scale=1 1 1; visual mesh filename=../meshes/qbhand/ph_short_yupzfront1.STL scale=1 1 1
- link left_qbhand_index_proximal_link: geometry collision mesh filename=../meshes/qbhand/ph_medium_yupzfront1.STL scale=1 1 1; visual mesh filename=../meshes/qbhand/ph_medium_yupzfront1.STL scale=1 1 1
- link left_qbhand_little_distal_link: geometry collision mesh filename=../meshes/qbhand/ph_distal_yupzfront1.STL scale=1 1 1; visual mesh filename=../meshes/qbhand/ph_distal_yupzfront1.STL scale=1 1 1
- link left_qbhand_little_knuckle_link: geometry collision mesh filename=../meshes/qbhand/ph_knuckle_yupzfront1.STL scale=1 1 1; visual mesh filename=../meshes/qbhand/ph_knuckle_yupzfront1.STL scale=1 1 1
- link left_qbhand_little_middle_link: geometry collision mesh filename=../meshes/qbhand/ph_short_yupzfront1.STL scale=1 1 1; visual mesh filename=../meshes/qbhand/ph_short_yupzfront1.STL scale=1 1 1
- link left_qbhand_little_proximal_link: geometry collision mesh filename=../meshes/qbhand/ph_short_yupzfront1.STL scale=1 1 1; visual mesh filename=../meshes/qbhand/ph_short_yupzfront1.STL scale=1 1 1
- link left_qbhand_middle_distal_link: geometry collision mesh filename=../meshes/qbhand/ph_distal_yupzfront1.STL scale=1 1 1; visual mesh filename=../meshes/qbhand/ph_distal_yupzfront1.STL scale=1 1 1
- link left_qbhand_middle_knuckle_link: geometry collision mesh filename=../meshes/qbhand/ph_knuckle_yupzfront1.STL scale=1 1 1; visual mesh filename=../meshes/qbhand/ph_knuckle_yupzfront1.STL scale=1 1 1
- link left_qbhand_middle_middle_link: geometry collision mesh filename=../meshes/qbhand/ph_short_yupzfront1.STL scale=1 1 1; visual mesh filename=../meshes/qbhand/ph_short_yupzfront1.STL scale=1 1 1
- link left_qbhand_middle_proximal_link: geometry collision mesh filename=../meshes/qbhand/ph_medium_yupzfront1.STL scale=1 1 1; visual mesh filename=../meshes/qbhand/ph_medium_yupzfront1.STL scale=1 1 1
- link left_qbhand_palm_link: geometry collision mesh filename=../meshes/qbhand/palm_pinch_l_yupzfront1.STL scale=1000 1000 1000; visual mesh filename=../meshes/qbhand/palm_pinch_l_yupzfront1.STL scale=1000 1000 1000
- link left_qbhand_ring_distal_link: geometry collision mesh filename=../meshes/qbhand/ph_distal_yupzfront1.STL scale=1 1 1; visual mesh filename=../meshes/qbhand/ph_distal_yupzfront1.STL scale=1 1 1
- link left_qbhand_ring_knuckle_link: geometry collision mesh filename=../meshes/qbhand/ph_knuckle_yupzfront1.STL scale=1 1 1; visual mesh filename=../meshes/qbhand/ph_knuckle_yupzfront1.STL scale=1 1 1
- link left_qbhand_ring_middle_link: geometry collision mesh filename=../meshes/qbhand/ph_short_yupzfront1.STL scale=1 1 1; visual mesh filename=../meshes/qbhand/ph_short_yupzfront1.STL scale=1 1 1
- link left_qbhand_ring_proximal_link: geometry collision mesh filename=../meshes/qbhand/ph_medium_yupzfront1.STL scale=1 1 1; visual mesh filename=../meshes/qbhand/ph_medium_yupzfront1.STL scale=1 1 1
- link left_qbhand_thumb_distal_link: geometry collision mesh filename=../meshes/qbhand/ph_distal_yupzfront1.STL scale=1 1 1; visual mesh filename=../meshes/qbhand/ph_distal_yupzfront1.STL scale=1 1 1
- link left_qbhand_thumb_knuckle_link: geometry collision mesh filename=../meshes/qbhand/ph_thumb_l_yupzfront1.STL scale=1 1 1; visual mesh filename=../meshes/qbhand/ph_thumb_l_yupzfront1.STL scale=1 1 1
- link left_qbhand_thumb_proximal_link: geometry collision mesh filename=../meshes/qbhand/ph_short_yupzfront1.STL scale=1 1 1; visual mesh filename=../meshes/qbhand/ph_short_yupzfront1.STL scale=1 1 1
- link right_qbhand_base_link: geometry collision mesh filename=../meshes/qbhand/flange_iso_04_yupzfront.STL scale=1 1 1; visual mesh filename=../meshes/qbhand/flange_iso_04_yupzfront.STL scale=1 1 1
- link right_qbhand_index_distal_link: geometry collision mesh filename=../meshes/qbhand/ph_distal_yupzfront1.STL scale=1 1 1; visual mesh filename=../meshes/qbhand/ph_distal_yupzfront1.STL scale=1 1 1
- link right_qbhand_index_knuckle_link: geometry collision mesh filename=../meshes/qbhand/ph_knuckle_yupzfront1.STL scale=1 1 1; visual mesh filename=../meshes/qbhand/ph_knuckle_yupzfront1.STL scale=1 1 1
- link right_qbhand_index_middle_link: geometry collision mesh filename=../meshes/qbhand/ph_short_yupzfront1.STL scale=1 1 1; visual mesh filename=../meshes/qbhand/ph_short_yupzfront1.STL scale=1 1 1
- link right_qbhand_index_proximal_link: geometry collision mesh filename=../meshes/qbhand/ph_medium_yupzfront1.STL scale=1 1 1; visual mesh filename=../meshes/qbhand/ph_medium_yupzfront1.STL scale=1 1 1
- link right_qbhand_little_distal_link: geometry collision mesh filename=../meshes/qbhand/ph_distal_yupzfront1.STL scale=1 1 1; visual mesh filename=../meshes/qbhand/ph_distal_yupzfront1.STL scale=1 1 1
- link right_qbhand_little_knuckle_link: geometry collision mesh filename=../meshes/qbhand/ph_knuckle_yupzfront1.STL scale=1 1 1; visual mesh filename=../meshes/qbhand/ph_knuckle_yupzfront1.STL scale=1 1 1
- link right_qbhand_little_middle_link: geometry collision mesh filename=../meshes/qbhand/ph_short_yupzfront1.STL scale=1 1 1; visual mesh filename=../meshes/qbhand/ph_short_yupzfront1.STL scale=1 1 1
- link right_qbhand_little_proximal_link: geometry collision mesh filename=../meshes/qbhand/ph_short_yupzfront1.STL scale=1 1 1; visual mesh filename=../meshes/qbhand/ph_short_yupzfront1.STL scale=1 1 1
- link right_qbhand_middle_distal_link: geometry collision mesh filename=../meshes/qbhand/ph_distal_yupzfront1.STL scale=1 1 1; visual mesh filename=../meshes/qbhand/ph_distal_yupzfront1.STL scale=1 1 1
- link right_qbhand_middle_knuckle_link: geometry collision mesh filename=../meshes/qbhand/ph_knuckle_yupzfront1.STL scale=1 1 1; visual mesh filename=../meshes/qbhand/ph_knuckle_yupzfront1.STL scale=1 1 1
- link right_qbhand_middle_middle_link: geometry collision mesh filename=../meshes/qbhand/ph_short_yupzfront1.STL scale=1 1 1; visual mesh filename=../meshes/qbhand/ph_short_yupzfront1.STL scale=1 1 1
- link right_qbhand_middle_proximal_link: geometry collision mesh filename=../meshes/qbhand/ph_medium_yupzfront1.STL scale=1 1 1; visual mesh filename=../meshes/qbhand/ph_medium_yupzfront1.STL scale=1 1 1
- link right_qbhand_palm_link: geometry collision mesh filename=../meshes/qbhand/palm_pinch_r.stl scale=0.001 0.001 0.001; visual mesh filename=../meshes/qbhand/palm_pinch_r_yupzfront2.STL scale=1 1 1
- link right_qbhand_ring_distal_link: geometry collision mesh filename=../meshes/qbhand/ph_distal_yupzfront1.STL scale=1 1 1; visual mesh filename=../meshes/qbhand/ph_distal_yupzfront1.STL scale=1 1 1
- link right_qbhand_ring_knuckle_link: geometry collision mesh filename=../meshes/qbhand/ph_knuckle_yupzfront1.STL scale=1 1 1; visual mesh filename=../meshes/qbhand/ph_knuckle_yupzfront1.STL scale=1 1 1
- link right_qbhand_ring_middle_link: geometry collision mesh filename=../meshes/qbhand/ph_short_yupzfront1.STL scale=1 1 1; visual mesh filename=../meshes/qbhand/ph_short_yupzfront1.STL scale=1 1 1
- link right_qbhand_ring_proximal_link: geometry collision mesh filename=../meshes/qbhand/ph_medium_yupzfront1.STL scale=1 1 1; visual mesh filename=../meshes/qbhand/ph_medium_yupzfront1.STL scale=1 1 1
- link right_qbhand_thumb_distal_link: geometry collision mesh filename=../meshes/qbhand/ph_distal_yupzfront1.STL scale=1 1 1; visual mesh filename=../meshes/qbhand/ph_distal_yupzfront1.STL scale=1 1 1
- link right_qbhand_thumb_knuckle_link: geometry collision mesh filename=../meshes/qbhand/ph_thumb_r_yupzfront1.STL scale=1 1 1; visual mesh filename=../meshes/qbhand/ph_thumb_r_yupzfront1.STL scale=1 1 1
- link right_qbhand_thumb_proximal_link: geometry collision mesh filename=../meshes/qbhand/ph_short_yupzfront1.STL scale=1 1 1; visual mesh filename=../meshes/qbhand/ph_short_yupzfront1.STL scale=1 1 1
- link torso_end: geometry collision mesh filename=../meshes/clover/collision/torso_end_v2_yup.STL; visual mesh filename=../meshes/clover/visual/torso_end_v2_yup.dae
Joints:
- joint left_qbhand_thumb_knuckle_joint: axis 0 0 -1 -> 0 0 1

File: rofunc/simulator/assets/urdf/curi/urdf/curi_yup.urdf (robot description, URDF)
Before this commit: robot curi, 41 links, 40 joints
Links:
- link torso_end: geometry collision mesh filename=../meshes/clover/collision/torso_end_v2_yup.stl; visual mesh filename=../meshes/clover/visual/torso_end_v2_yup.dae
