Commit message: Update curi dual arm model

File: rofunc/simulator/assets/urdf/curi/urdf/curi_isaacgym_dual_arm.urdf (robot description, URDF)
Before this commit: robot curi, 39 links, 38 joints
Links:
- link torso_end: geometry collision mesh filename=../meshes/clover/collision/torso_end_v2_yup.stl; visual mesh filename=../meshes/clover/visual/torso_end_v2_yup.dae
Joints:
- joint head_joint_torso_end: origin xyz=0.01466 0 0.2775 rpy=0 0 0 -> xyz=0.02 0 0.3929 rpy=0 0 0
- joint panda_left_joint_torso_end: origin xyz=0.02842 0.11216 0.19004 rpy=-1.5004311592913677 0.8772798703277918 -0.2038499389018784 -> xyz=-0.08537 0.07009 0.2535 rpy=-1.3685238493647454 0.913218224774749 -0.6168337646727412
- joint panda_right_joint_torso_end: origin xyz=0.02842 -0.11216 0.19004 rpy=1.5004311592913677 0.8772798703277918 0.2038499389018784 -> xyz=-0.08537 -0.07009 0.2535 rpy=1.3685238493647454 0.913218224774749 0.6168337646727412
