Commit message: Add Torso Shell

File: rofunc/simulator/assets/urdf/curi/urdf/curi.urdf (robot description, URDF)
Before this commit: robot curi, 41 links, 40 joints
Links:
- added link shell, mass 1.63531; collision mesh filename=../meshes/clover/collision/Shell_v2_Share_zup.STL; visual mesh filename=../meshes/clover/visual/Shell_v2_Share_zup.dae
Joints:
- added joint shell_torso_end: type fixed, parent torso_end, child shell, origin xyz=0 0 0 rpy=0 0 0

File: rofunc/simulator/assets/urdf/curi/urdf/curi_isaacgym.urdf (robot description, URDF)
Before this commit: robot curi, 39 links, 38 joints
Links:
- added link shell, mass 1.63531; collision mesh filename=../meshes/clover/collision/Shell_v2_Share_yup.STL; visual mesh filename=../meshes/clover/visual/Shell_v2_Share_yup.dae
Joints:
- added joint shell_torso_end: type fixed, parent torso_end, child shell, origin xyz=0 0 0 rpy=0 0 0

File: rofunc/simulator/assets/urdf/curi/urdf/curi_w_softhand.urdf (robot description, URDF)
Before this commit: robot curi, 111 links, 110 joints
Links:
- added link shell, mass 1.63531; collision mesh filename=../meshes/clover/collision/Shell_v2_Share_zup.STL; visual mesh filename=../meshes/clover/visual/Shell_v2_Share_zup.dae
Joints:
- added joint shell_torso_end: type fixed, parent torso_end, child shell, origin xyz=0 0 0 rpy=0 0 0

File: rofunc/simulator/assets/urdf/curi/urdf/curi_w_softhand_isaacgym.urdf (robot description, URDF)
Before this commit: robot curi, 109 links, 108 joints
Links:
- added link shell, mass 1.63531; collision mesh filename=../meshes/clover/collision/Shell_v2_Share_yup.STL; visual mesh filename=../meshes/clover/visual/Shell_v2_Share_yup.dae
- link torso_end: geometry collision mesh filename=../meshes/clover/collision/torso_end_v2_yup.STL; visual mesh filename=../meshes/clover/visual/torso_end_v2_yup.dae
Joints:
- added joint shell_torso_end: type fixed, parent torso_end, child shell, origin xyz=0 0 0 rpy=0 0 0

File: rofunc/simulator/assets/urdf/curi/urdf/curi_w_softhand_yup.urdf (robot description, URDF)
Before this commit: robot curi, 111 links, 110 joints
Links:
- added link shell, mass 1.63531; collision mesh filename=../meshes/clover/collision/Shell_v2_Share_yup.STL; visual mesh filename=../meshes/clover/visual/Shell_v2_Share_yup.dae
Joints:
- added joint shell_torso_end: type fixed, parent torso_end, child shell, origin xyz=0 0 0 rpy=0 0 0

File: rofunc/simulator/assets/urdf/curi/urdf/curi_yup.urdf (robot description, URDF)
Before this commit: robot curi, 41 links, 40 joints
Links:
- added link shell, mass 1.63531; collision mesh filename=../meshes/clover/collision/Shell_v2_Share_yup.STL; visual mesh filename=../meshes/clover/visual/Shell_v2_Share_yup.dae
Joints:
- added joint shell_torso_end: type fixed, parent torso_end, child shell, origin xyz=0 0 0 rpy=0 0 0
