Commit message: 🚀🎉 [RofuncRL] Image obs is available for IsaacGym RL tasks

File: rofunc/simulator/assets/urdf/curi/urdf/curi_isaacgym_dual_arm_w_head.urdf (robot description, URDF)
Before this commit: robot curi, 40 links, 39 joints
Joints:
- joint head_actuated_joint1: type fixed -> revolute
- joint head_actuated_joint2: type fixed -> revolute
