Commit message: Added 90 degree flange to qbhand

File: rofunc/simulator/assets/urdf/curi/urdf/curi_w_softhand.urdf (robot description, URDF)
Before this commit: robot curi, 112 links, 111 joints
Links:
- added link flange90_l; collision mesh filename=../meshes/clover/visual/flange90_zup.STL; visual mesh filename=../meshes/clover/visual/flange90_zup.dae
- added link flange90_r; collision mesh filename=../meshes/clover/visual/flange90_zup.STL; visual mesh filename=../meshes/clover/visual/flange90_zup.dae
Joints:
- added joint left_qbhand_flange_joint: type fixed, parent left_hand_root_link, child flange90_l, origin xyz=0 0 0 rpy=0 0 0.7854
- added joint right_qbhand_flange_joint: type fixed, parent right_hand_root_link, child flange90_r, origin xyz=0 0 0 rpy=0 0 -2.3562
- joint left_qbhand_base_fixed_joint: origin xyz=0 0 0 rpy=0 0 0 -> xyz=0.046 0 0.038 rpy=1.5708 0 1.5708; parent left_hand_root_link -> flange90_l
- joint right_qbhand_base_fixed_joint: origin xyz=0 0 0 rpy=0 0 0 -> xyz=0.046 0 0.038 rpy=1.5708 0 1.5708; parent right_hand_root_link -> flange90_r

File: rofunc/simulator/assets/urdf/curi/urdf/curi_w_softhand_isaacgym.urdf (robot description, URDF)
Before this commit: robot curi, 110 links, 109 joints
Links:
- added link flange90_l; collision mesh filename=../meshes/clover/visual/flange90_yup.STL; visual mesh filename=../meshes/clover/visual/flange90_yup.dae
- added link flange90_r; collision mesh filename=../meshes/clover/visual/flange90_yup.STL; visual mesh filename=../meshes/clover/visual/flange90_yup.dae
Joints:
- added joint left_qbhand_flange_joint: type fixed, parent left_hand_root_link, child flange90_l, origin xyz=0 0 0 rpy=0 0 0.7854
- added joint right_qbhand_flange_joint: type fixed, parent right_hand_root_link, child flange90_r, origin xyz=0 0 0 rpy=0 0 -2.3562
- joint left_qbhand_base_fixed_joint: origin xyz=0 0 0 rpy=0 0 0 -> xyz=0.046 0 0.038 rpy=1.5708 0 1.5708; parent left_hand_root_link -> flange90_l
- joint right_qbhand_base_fixed_joint: origin xyz=0 0 0 rpy=0 0 0 -> xyz=0.046 0 0.038 rpy=1.5708 0 1.5708; parent right_hand_root_link -> flange90_r

File: rofunc/simulator/assets/urdf/curi/urdf/curi_w_softhand_yup.urdf (robot description, URDF)
Before this commit: robot curi, 112 links, 111 joints
Links:
- added link flange90_l; collision mesh filename=../meshes/clover/visual/flange90_yup.STL; visual mesh filename=../meshes/clover/visual/flange90_yup.dae
- added link flange90_r; collision mesh filename=../meshes/clover/visual/flange90_yup.STL; visual mesh filename=../meshes/clover/visual/flange90_yup.dae
Joints:
- added joint left_qbhand_flange_joint: type fixed, parent left_hand_root_link, child flange90_l, origin xyz=0 0 0 rpy=0 0 0.7854
- added joint right_qbhand_flange_joint: type fixed, parent right_hand_root_link, child flange90_r, origin xyz=0 0 0 rpy=0 0 -2.3562
- joint left_qbhand_base_fixed_joint: origin xyz=0 0 0 rpy=0 0 0 -> xyz=0.046 0 0.038 rpy=1.5708 0 1.5708; parent left_hand_root_link -> flange90_l
- joint right_qbhand_base_fixed_joint: origin xyz=0 0 0 rpy=0 0 0 -> xyz=0.046 0 0.038 rpy=1.5708 0 1.5708; parent right_hand_root_link -> flange90_r

Commit message: Add files via upload
fixed right flange angle problem

File: rofunc/simulator/assets/urdf/curi/urdf/curi_w_softhand.urdf (robot description, URDF)
Before this commit: robot curi, 114 links, 113 joints
Joints:
- joint right_qbhand_flange_joint: origin xyz=0 0 0 rpy=0 0 -2.3562 -> xyz=0 0 0 rpy=0 0 -0.7855

File: rofunc/simulator/assets/urdf/curi/urdf/curi_w_softhand_isaacgym.urdf (robot description, URDF)
Before this commit: robot curi, 112 links, 111 joints
Joints:
- joint right_qbhand_flange_joint: origin xyz=0 0 0 rpy=0 0 -2.3562 -> xyz=0 0 0 rpy=0 0 -0.7855

File: rofunc/simulator/assets/urdf/curi/urdf/curi_w_softhand_yup.urdf (robot description, URDF)
Before this commit: robot curi, 114 links, 113 joints
Joints:
- joint right_qbhand_flange_joint: origin xyz=0 0 0 rpy=0 0 -2.3562 -> xyz=0 0 0 rpy=0 0 -0.7855
