Commit message: 🎮 Add hotu_humanoid_w_hand MJCF model

File: rofunc/simulator/assets/urdf/curi/urdf/qbhand_left.urdf (robot description, URDF)
Before this commit: robot qbhand, 38 links, 37 joints
Links:
- link qbhand_base_link: geometry collision mesh filename=../meshes/qbhand/flange_iso_04.stl scale=0.001 0.001 0.001; visual mesh filename=../meshes/qbhand/flange_iso_04.stl scale=0.001 0.001 0.001
- link qbhand_index_distal_link: geometry collision mesh filename=../meshes/qbhand/ph_distal_collision.stl scale=0.001 0.001 0.001; visual mesh filename=../meshes/qbhand/ph_distal.stl scale=0.001 0.001 0.001
- link qbhand_index_knuckle_link: geometry collision mesh filename=../meshes/qbhand/ph_knuckle_collision.stl scale=0.001 0.001 0.001; visual mesh filename=../meshes/qbhand/ph_knuckle.stl scale=0.001 0.001 0.001
- link qbhand_index_middle_link: geometry collision mesh filename=../meshes/qbhand/ph_short_collision.stl scale=0.001 0.001 0.001; visual mesh filename=../meshes/qbhand/ph_short.stl scale=0.001 0.001 0.001
- link qbhand_index_proximal_link: geometry collision mesh filename=../meshes/qbhand/ph_medium_collision.stl scale=0.001 0.001 0.001; visual mesh filename=../meshes/qbhand/ph_medium.stl scale=0.001 0.001 0.001
- link qbhand_little_distal_link: geometry collision mesh filename=../meshes/qbhand/ph_distal_collision.stl scale=0.001 0.001 0.001; visual mesh filename=../meshes/qbhand/ph_distal.stl scale=0.001 0.001 0.001
- link qbhand_little_knuckle_link: geometry collision mesh filename=../meshes/qbhand/ph_knuckle_collision.stl scale=0.001 0.001 0.001; visual mesh filename=../meshes/qbhand/ph_knuckle.stl scale=0.001 0.001 0.001
- link qbhand_little_middle_link: geometry collision mesh filename=../meshes/qbhand/ph_short_collision.stl scale=0.001 0.001 0.001; visual mesh filename=../meshes/qbhand/ph_short.stl scale=0.001 0.001 0.001
- link qbhand_little_proximal_link: geometry collision mesh filename=../meshes/qbhand/ph_short_collision.stl scale=0.001 0.001 0.001; visual mesh filename=../meshes/qbhand/ph_short.stl scale=0.001 0.001 0.001
- link qbhand_middle_distal_link: geometry collision mesh filename=../meshes/qbhand/ph_distal_collision.stl scale=0.001 0.001 0.001; visual mesh filename=../meshes/qbhand/ph_distal.stl scale=0.001 0.001 0.001
- link qbhand_middle_knuckle_link: geometry collision mesh filename=../meshes/qbhand/ph_knuckle_collision.stl scale=0.001 0.001 0.001; visual mesh filename=../meshes/qbhand/ph_knuckle.stl scale=0.001 0.001 0.001
- link qbhand_middle_middle_link: geometry collision mesh filename=../meshes/qbhand/ph_short_collision.stl scale=0.001 0.001 0.001; visual mesh filename=../meshes/qbhand/ph_short.stl scale=0.001 0.001 0.001
- link qbhand_middle_proximal_link: geometry collision mesh filename=../meshes/qbhand/ph_medium_collision.stl scale=0.001 0.001 0.001; visual mesh filename=../meshes/qbhand/ph_medium.stl scale=0.001 0.001 0.001
- link qbhand_palm_link: geometry collision mesh filename=../meshes/qbhand/palm_pinch_l.stl scale=0.001 0.001 0.001; visual mesh filename=../meshes/qbhand/palm_pinch_l.stl scale=0.001 0.001 0.001
- link qbhand_ring_distal_link: geometry collision mesh filename=../meshes/qbhand/ph_distal_collision.stl scale=0.001 0.001 0.001; visual mesh filename=../meshes/qbhand/ph_distal.stl scale=0.001 0.001 0.001
- link qbhand_ring_knuckle_link: geometry collision mesh filename=../meshes/qbhand/ph_knuckle_collision.stl scale=0.001 0.001 0.001; visual mesh filename=../meshes/qbhand/ph_knuckle.stl scale=0.001 0.001 0.001
- link qbhand_ring_middle_link: geometry collision mesh filename=../meshes/qbhand/ph_short_collision.stl scale=0.001 0.001 0.001; visual mesh filename=../meshes/qbhand/ph_short.stl scale=0.001 0.001 0.001
- link qbhand_ring_proximal_link: geometry collision mesh filename=../meshes/qbhand/ph_medium_collision.stl scale=0.001 0.001 0.001; visual mesh filename=../meshes/qbhand/ph_medium.stl scale=0.001 0.001 0.001
- link qbhand_thumb_distal_link: geometry collision mesh filename=../meshes/qbhand/ph_distal_collision.stl scale=0.001 0.001 0.001; visual mesh filename=../meshes/qbhand/ph_distal.stl scale=0.001 0.001 0.001
- link qbhand_thumb_knuckle_link: geometry collision mesh filename=../meshes/qbhand/ph_thumb_l_collision.stl scale=0.001 0.001 0.001; visual mesh filename=../meshes/qbhand/ph_thumb_l.stl scale=0.001 0.001 0.001
- link qbhand_thumb_proximal_link: geometry collision mesh filename=../meshes/qbhand/ph_short_collision.stl scale=0.001 0.001 0.001; visual mesh filename=../meshes/qbhand/ph_short.stl scale=0.001 0.001 0.001

File: rofunc/simulator/assets/urdf/curi/urdf/qbhand_right.urdf (robot description, URDF)
Before this commit: robot qbhand, 38 links, 37 joints
Links:
- link qbhand_base_link: geometry collision mesh filename=../meshes/qbhand/flange_iso_04.stl scale=0.001 0.001 0.001; visual mesh filename=../meshes/qbhand/flange_iso_04.stl scale=0.001 0.001 0.001
- link qbhand_index_distal_link: geometry collision mesh filename=../meshes/qbhand/ph_distal_collision.stl scale=0.001 0.001 0.001; visual mesh filename=../meshes/qbhand/ph_distal.stl scale=0.001 0.001 0.001
- link qbhand_index_knuckle_link: geometry collision mesh filename=../meshes/qbhand/ph_knuckle_collision.stl scale=0.001 0.001 0.001; visual mesh filename=../meshes/qbhand/ph_knuckle.stl scale=0.001 0.001 0.001
- link qbhand_index_middle_link: geometry collision mesh filename=../meshes/qbhand/ph_short_collision.stl scale=0.001 0.001 0.001; visual mesh filename=../meshes/qbhand/ph_short.stl scale=0.001 0.001 0.001
- link qbhand_index_proximal_link: geometry collision mesh filename=../meshes/qbhand/ph_medium_collision.stl scale=0.001 0.001 0.001; visual mesh filename=../meshes/qbhand/ph_medium.stl scale=0.001 0.001 0.001
- link qbhand_little_distal_link: geometry collision mesh filename=../meshes/qbhand/ph_distal_collision.stl scale=0.001 0.001 0.001; visual mesh filename=../meshes/qbhand/ph_distal.stl scale=0.001 0.001 0.001
- link qbhand_little_knuckle_link: geometry collision mesh filename=../meshes/qbhand/ph_knuckle_collision.stl scale=0.001 0.001 0.001; visual mesh filename=../meshes/qbhand/ph_knuckle.stl scale=0.001 0.001 0.001
- link qbhand_little_middle_link: geometry collision mesh filename=../meshes/qbhand/ph_short_collision.stl scale=0.001 0.001 0.001; visual mesh filename=../meshes/qbhand/ph_short.stl scale=0.001 0.001 0.001
- link qbhand_little_proximal_link: geometry collision mesh filename=../meshes/qbhand/ph_short_collision.stl scale=0.001 0.001 0.001; visual mesh filename=../meshes/qbhand/ph_short.stl scale=0.001 0.001 0.001
- link qbhand_middle_distal_link: geometry collision mesh filename=../meshes/qbhand/ph_distal_collision.stl scale=0.001 0.001 0.001; visual mesh filename=../meshes/qbhand/ph_distal.stl scale=0.001 0.001 0.001
- link qbhand_middle_knuckle_link: geometry collision mesh filename=../meshes/qbhand/ph_knuckle_collision.stl scale=0.001 0.001 0.001; visual mesh filename=../meshes/qbhand/ph_knuckle.stl scale=0.001 0.001 0.001
- link qbhand_middle_middle_link: geometry collision mesh filename=../meshes/qbhand/ph_short_collision.stl scale=0.001 0.001 0.001; visual mesh filename=../meshes/qbhand/ph_short.stl scale=0.001 0.001 0.001
- link qbhand_middle_proximal_link: geometry collision mesh filename=../meshes/qbhand/ph_medium_collision.stl scale=0.001 0.001 0.001; visual mesh filename=../meshes/qbhand/ph_medium.stl scale=0.001 0.001 0.001
- link qbhand_palm_link: geometry collision mesh filename=../meshes/qbhand/palm_pinch_r.stl scale=0.001 0.001 0.001; visual mesh filename=../meshes/qbhand/palm_pinch_r.stl scale=0.001 0.001 0.001
- link qbhand_ring_distal_link: geometry collision mesh filename=../meshes/qbhand/ph_distal_collision.stl scale=0.001 0.001 0.001; visual mesh filename=../meshes/qbhand/ph_distal.stl scale=0.001 0.001 0.001
- link qbhand_ring_knuckle_link: geometry collision mesh filename=../meshes/qbhand/ph_knuckle_collision.stl scale=0.001 0.001 0.001; visual mesh filename=../meshes/qbhand/ph_knuckle.stl scale=0.001 0.001 0.001
- link qbhand_ring_middle_link: geometry collision mesh filename=../meshes/qbhand/ph_short_collision.stl scale=0.001 0.001 0.001; visual mesh filename=../meshes/qbhand/ph_short.stl scale=0.001 0.001 0.001
- link qbhand_ring_proximal_link: geometry collision mesh filename=../meshes/qbhand/ph_medium_collision.stl scale=0.001 0.001 0.001; visual mesh filename=../meshes/qbhand/ph_medium.stl scale=0.001 0.001 0.001
- link qbhand_thumb_distal_link: geometry collision mesh filename=../meshes/qbhand/ph_distal_collision.stl scale=0.001 0.001 0.001; visual mesh filename=../meshes/qbhand/ph_distal.stl scale=0.001 0.001 0.001
- link qbhand_thumb_knuckle_link: geometry collision mesh filename=../meshes/qbhand/ph_thumb_r_collision.stl scale=0.001 0.001 0.001; visual mesh filename=../meshes/qbhand/ph_thumb_r.stl scale=0.001 0.001 0.001
- link qbhand_thumb_proximal_link: geometry collision mesh filename=../meshes/qbhand/ph_short_collision.stl scale=0.001 0.001 0.001; visual mesh filename=../meshes/qbhand/ph_short.stl scale=0.001 0.001 0.001
