Commit message: 🎮 Update CURI and walker models

File: rofunc/simulator/assets/urdf/curi/urdf/curi_w_softhand_isaacgym.urdf (robot description, URDF)
Before this commit: robot curi, 112 links, 111 joints
Links:
- link flange90_r: geometry collision mesh filename=../meshes/clover/visual/flange90_yup.stl; visual mesh filename=../meshes/clover/visual/flange90_yup.dae
- link torso_end: geometry collision mesh filename=../meshes/clover/collision/torso_end_v2_yup.stl; visual mesh filename=../meshes/clover/visual/torso_end_v2_yup.dae

File: rofunc/simulator/assets/urdf/curi/urdf/curi_w_softhand_isaacgym_stir_fry.urdf (robot description, URDF)
Before this commit: robot curi, 114 links, 113 joints
Links:
- link flange90_l: geometry collision mesh filename=../meshes/clover/collision/flange90_yup.STL; visual mesh filename=../meshes/clover/visual/flange90_yup.dae
- link flange90_r: geometry collision mesh filename=../meshes/clover/collision/flange90_yup.STL; visual mesh filename=../meshes/clover/visual/flange90_yup.dae
- link torso_end: geometry collision mesh filename=../meshes/clover/collision/torso_end_v2_yup.stl; visual mesh filename=../meshes/clover/visual/torso_end_v2_yup.dae

File: rofunc/simulator/assets/urdf/walker/urdf/walker_cartesio_stir_fry.urdf (robot description, URDF)
Before this commit: robot walker, 48 links, 47 joints
Joints:
- joint left_limb_j7: limit lower=-0.3508 upper=0.3508 effort=2.5 velocity=3.1416 -> (none)
- joint right_limb_j7: limit lower=-0.3508 upper=0.3508 effort=2.5 velocity=3.1416 -> (none)

Commit message: 🚀 [RofuncRL] QbSoftHand model ok for learning tasks

File: rofunc/simulator/assets/urdf/curi/urdf/curi_w_softhand_isaacgym.urdf (robot description, URDF)
Before this commit: robot curi, 112 links, 111 joints
Links:
- link flange90_l: geometry collision mesh filename=../meshes/clover/collision/flange90_yup.STL; visual mesh filename=../meshes/clover/visual/flange90_yup.dae
- link flange90_r: geometry collision mesh filename=../meshes/clover/collision/flange90_yup.STL; visual mesh filename=../meshes/clover/visual/flange90_yup.dae
