Commit message: 🎮 CURI robot low-level API for LLM agent

File: rofunc/simulator/assets/urdf/curi/urdf/curi_isaacgym_fixed_torso.urdf (robot description, URDF)
Before this commit: robot curi, 40 links, 39 joints
Links:
- link summit_xls_base_link: mass 300.0 -> 125.0
Joints:
- joint torso_actuated_joint1: type revolute -> fixed

Commit message: 🚀 [RofuncRL] Add ShadowHand and QbSofthand Grasping Tasks

File: rofunc/simulator/assets/urdf/curi/urdf/curi_isaacgym_fixed_torso.urdf (robot description, URDF)
Before this commit: robot curi, 40 links, 39 joints
Joints:
- joint panda_left_joint1: limit lower=-2.8973 upper=2.8973 effort=87 velocity=2.1750 -> lower=-2.8973 upper=2.8973 effort=500 velocity=2.1750
- joint panda_left_joint2: limit lower=-1.7628 upper=1.7628 effort=87 velocity=2.1750 -> lower=-1.7628 upper=1.7628 effort=500 velocity=2.1750
- joint panda_left_joint3: limit lower=-2.8973 upper=2.8973 effort=87 velocity=2.1750 -> lower=-2.8973 upper=2.8973 effort=500 velocity=2.1750
- joint panda_left_joint4: limit lower=-3.0718 upper=-0.0698 effort=87 velocity=2.1750 -> lower=-3.0718 upper=-0.0698 effort=500 velocity=2.1750
- joint panda_left_joint5: limit lower=-2.8973 upper=2.8973 effort=12 velocity=2.6100 -> lower=-2.8973 upper=2.8973 effort=500 velocity=2.6100
- joint panda_left_joint6: limit lower=-0.0175 upper=3.7525 effort=12 velocity=2.6100 -> lower=-0.0175 upper=3.7525 effort=500 velocity=2.6100
- joint panda_left_joint7: limit lower=-2.8973 upper=2.8973 effort=12 velocity=2.6100 -> lower=-2.8973 upper=2.8973 effort=500 velocity=2.6100
- joint panda_right_joint1: limit lower=-2.8973 upper=2.8973 effort=87 velocity=2.1750 -> lower=-2.8973 upper=2.8973 effort=500 velocity=2.1750
- joint panda_right_joint2: limit lower=-1.7628 upper=1.7628 effort=87 velocity=2.1750 -> lower=-1.7628 upper=1.7628 effort=500 velocity=2.1750
- joint panda_right_joint3: limit lower=-2.8973 upper=2.8973 effort=87 velocity=2.1750 -> lower=-2.8973 upper=2.8973 effort=500 velocity=2.1750
- joint panda_right_joint4: limit lower=-3.0718 upper=-0.0698 effort=87 velocity=2.1750 -> lower=-3.0718 upper=-0.0698 effort=500 velocity=2.1750
- joint panda_right_joint5: limit lower=-2.8973 upper=2.8973 effort=12 velocity=2.6100 -> lower=-2.8973 upper=2.8973 effort=500 velocity=2.6100
- joint panda_right_joint6: limit lower=-0.0175 upper=3.7525 effort=12 velocity=2.6100 -> lower=-0.0175 upper=3.7525 effort=500 velocity=2.6100
- joint panda_right_joint7: limit lower=-2.8973 upper=2.8973 effort=12 velocity=2.6100 -> lower=-2.8973 upper=2.8973 effort=500 velocity=2.6100
