Commit message: fix the bug

File: rofunc/simulator/assets/urdf/sektion_cabinet_model/urdf/sektion_cabinet.urdf (robot description, URDF)
Before this commit: robot cabinet_sektion, 9 links, 8 joints
Links:
- link door_left_link: geometry collision mesh filename=../meshes/door_left.stl scale=1.0 1.0 1.0; visual mesh filename=../meshes/door_left.obj scale=1.0 1.0 1.0
- link door_left_nob_link: geometry collision mesh filename=../meshes/door_left_nob.stl scale=1.0 1.0 1.0; visual mesh filename=../meshes/door_left_nob.obj scale=1.0 1.0 1.0
- link door_right_link: geometry collision mesh filename=../meshes/door_right.stl scale=1.0 1.0 1.0; visual mesh filename=../meshes/door_right.obj scale=1.0 1.0 1.0
- link door_right_nob_link: geometry collision mesh filename=../meshes/door_right_nob.stl scale=1.0 1.0 1.0; visual mesh filename=../meshes/door_right_nob.obj scale=1.0 1.0 1.0
- link drawer_bottom: geometry collision mesh filename=../meshes/drawer_convexdecomposition.obj scale=1.0 1.0 1.0; visual mesh filename=../meshes/drawer.obj scale=1.0 1.0 1.0
- link drawer_handle_bottom: geometry collision mesh filename=../meshes/drawer_handle_convexdecomposition.obj scale=1.0 1.0 1.0; visual mesh filename=../meshes/drawer_handle.obj scale=1.0 1.0 1.0
- link drawer_handle_top: geometry collision box size=0.014 0.02 0.15; collision box size=0.04 0.02 0.005
- link drawer_top: geometry collision mesh filename=../meshes/drawer_convexdecomposition.obj scale=1.0 1.0 1.0; visual mesh filename=../meshes/drawer.obj scale=1.0 1.0 1.0
- link sektion: geometry collision mesh filename=../meshes/sektion_convexdecomposition.obj scale=1.0 1.0 1.0; visual mesh filename=../meshes/sektion.obj scale=1.0 1.0 1.0

File: rofunc/simulator/assets/urdf/sektion_cabinet_model/urdf/sektion_cabinet_2.urdf (robot description, URDF)
Before this commit: robot cabinet_sektion, 9 links, 8 joints
Links:
- link door_left_link: geometry collision mesh filename=../meshes/door_left.stl scale=1.0 1.0 1.0; visual mesh filename=../meshes/door_left.obj scale=1.0 1.0 1.0
- link door_left_nob_link: geometry collision mesh filename=../meshes/door_left_nob.stl scale=1.0 1.0 1.0; visual mesh filename=../meshes/door_left_nob.obj scale=1.0 1.0 1.0
- link door_right_link: geometry collision mesh filename=../meshes/door_right.stl scale=1.0 1.0 1.0; visual mesh filename=../meshes/door_right.obj scale=1.0 1.0 1.0
- link door_right_nob_link: geometry collision mesh filename=../meshes/door_right_nob.stl scale=1.0 1.0 1.0; visual mesh filename=../meshes/door_right_nob.obj scale=1.0 1.0 1.0
- link drawer_bottom: geometry collision mesh filename=../meshes/drawer_convexdecomposition.obj scale=1.0 1.0 1.0; visual mesh filename=../meshes/drawer.obj scale=1.0 1.0 1.0
- link drawer_handle_bottom: geometry collision mesh filename=../meshes/drawer_handle_convexdecomposition.obj scale=1.0 1.0 1.0; visual mesh filename=../meshes/drawer_handle.obj scale=1.0 1.0 1.0
- link drawer_handle_top: geometry collision mesh filename=../meshes/drawer_handle_convexdecomposition.obj scale=1.0 1.0 1.0; visual mesh filename=../meshes/drawer_handle.obj scale=1.0 1.0 1.0
- link drawer_top: geometry collision mesh filename=../meshes/drawer_convexdecomposition0.obj scale=1.0 1.0 1.0; collision mesh filename=../meshes/drawer_convexdecomposition1.obj scale=1.0 1.0 1.0
- link sektion: geometry collision mesh filename=../meshes/sektion_convexdecomposition0.obj scale=1.0 1.0 1.0; collision mesh filename=../meshes/sektion_convexdecomposition1.obj scale=1.0 1.0 1.0
