Commit message: Add two examples for walker and diablo

File: rofunc/simulator/assets/urdf/walker/urdf/walker.urdf (robot description, URDF)
Before this commit: robot walker, 63 links, 62 joints
Links:
- added link world
Joints:
- added joint reference: type floating, parent world, child base_link
- joint right_pinky_j1: limit lower=0 upper=1.5708 effort=0 velocity=0 -> lower=0 upper=1.5708 effort= velocity=0

Commit message: Update walker sim

File: rofunc/simulator/assets/urdf/walker/urdf/walker.urdf (robot description, URDF)
Before this commit: robot walker, 64 links, 63 joints
Links:
- added link right_elbow
Joints:
- added joint right_elbow_joint: type fixed, parent right_limb_l4, child right_elbow, origin xyz=0 0 0 rpy=0 -1.5708 -3.1416, axis 0 0 1
- joint right_pinky_j1: limit lower=0 upper=1.5708 effort= velocity=0 -> lower=0 upper=1.5708 effort=0 velocity=0

File: rofunc/simulator/assets/urdf/walker/urdf/walker_ct_lower.urdf (robot description, URDF)
Before this commit: robot walker, 17 links, 16 joints
Links:
- link left_leg_l1: geometry collision mesh filename=../meshes/left_leg_l1.STL; visual mesh filename=../meshes/left_leg_l1.STL
- link left_leg_l2: geometry collision mesh filename=../meshes/left_leg_l2.STL; visual mesh filename=../meshes/left_leg_l2.STL
- link left_leg_l3: geometry collision mesh filename=../meshes/left_leg_l3.STL; visual mesh filename=../meshes/left_leg_l3.STL
- link left_leg_l4: geometry collision mesh filename=../meshes/left_leg_l4.STL; visual mesh filename=../meshes/left_leg_l4.STL
- link left_leg_l5: geometry collision mesh filename=../meshes/left_leg_l5.STL; visual mesh filename=../meshes/left_leg_l5.STL
- link left_leg_l6: geometry collision mesh filename=../meshes/left_leg_l6.STL; visual mesh filename=../meshes/left_leg_l6.STL
- link left_leg_link1: geometry collision mesh filename=../meshes/left_leg_link1.STL; visual mesh filename=../meshes/left_leg_link1.STL
- link left_leg_link2: geometry collision mesh filename=../meshes/left_leg_link2.STL; visual mesh filename=../meshes/left_leg_link2.STL
- link right_leg_l1: geometry collision mesh filename=../meshes/right_leg_l1.STL; visual mesh filename=../meshes/right_leg_l1.STL
- link right_leg_l2: geometry collision mesh filename=../meshes/right_leg_l2.STL; visual mesh filename=../meshes/right_leg_l2.STL
- link right_leg_l3: geometry collision mesh filename=../meshes/right_leg_l3.STL; visual mesh filename=../meshes/right_leg_l3.STL
- link right_leg_l4: geometry collision mesh filename=../meshes/right_leg_l4.STL; visual mesh filename=../meshes/right_leg_l4.STL
- link right_leg_l5: geometry collision mesh filename=../meshes/right_leg_l5.STL; visual mesh filename=../meshes/right_leg_l5.STL
- link right_leg_l6: geometry collision mesh filename=../meshes/right_leg_l6.STL; visual mesh filename=../meshes/right_leg_l6.STL
- link right_leg_link1: geometry collision mesh filename=../meshes/right_leg_link1.STL; visual mesh filename=../meshes/right_leg_link1.STL
- link right_leg_link2: geometry collision mesh filename=../meshes/right_leg_link2.STL; visual mesh filename=../meshes/right_leg_link2.STL
- link torso: geometry collision mesh filename=../meshes/base_link.STL; visual mesh filename=../meshes/base_link.STL
