Commit message: 🎮 Update simulator
Plan to refactor codes in the simulator

File: rofunc/simulator/assets/urdf/walker/urdf/walker_cartesio_stir_fry.urdf (robot description, URDF)
Before this commit: robot walker, 48 links, 47 joints
Links:
- link pan_link: geometry collision mesh filename=../../objects/pan_spoon/pan.obj scale=1 1 -1; visual mesh filename=../../objects/pan_spoon/pan.obj scale=1 1 -1
- link spoon_link: geometry collision mesh filename=../../objects/pan_spoon/spoon.obj scale=-1 1 1; visual mesh filename=../../objects/pan_spoon/spoon.obj scale=-1 1 1
Joints:
- joint left_pan_joint: origin xyz=-0.02 -0.06 0.017 rpy=-1.27 -1.57 1.57 -> xyz=0 0 0 rpy=0 -0.8 -1.9
- joint right_spoon_joint: origin xyz=0.02 -0.05 0.04 rpy=-1.57 -1.57 -1.87 -> xyz=0 0 0 rpy=1 -0.3 1.5
