Commit message: Update data

File: rofunc/simulator/assets/urdf/human/human_xsenstemplate_48dof_zxy.urdf (robot description, URDF)
Before this commit: robot XSensStyleModel_template, 49 links, 48 joints
Joints:
- joint jLeftC7Shoulder_rotx: axis 1 0 0 -> -1 0 0
- joint jLeftElbow_roty: axis 0 1 0 -> 0 0 -1
- joint jLeftElbow_rotz: axis 0 0 1 -> 0 -1 0
- joint jLeftShoulder_rotx: axis 1 0 0 -> -1 0 0; origin xyz=0 0 0 rpy=0 0 0 -> xyz=0 0 0 rpy=-1.5 0 0
- joint jLeftShoulder_roty: axis 0 1 0 -> 0 0 -1
- joint jLeftShoulder_rotz: axis 0 0 1 -> 0 -1 0
- joint jLeftWrist_rotx: axis 1 0 0 -> -1 0 0
- joint jLeftWrist_rotz: axis 0 0 1 -> 0 -1 0
- joint jRightAnkle_rotx: axis 1 0 0 -> -1 0 0
- joint jRightAnkle_roty: axis 0 1 0 -> 0 0 -1
- joint jRightAnkle_rotz: axis 0 0 1 -> 0 -1 0
- joint jRightBallFoot_roty: axis 0 1 0 -> 0 0 -1
- joint jRightElbow_roty: axis 0 1 0 -> 0 0 1
- joint jRightElbow_rotz: axis 0 0 1 -> 0 -1 0
- joint jRightHip_rotx: axis 1 0 0 -> -1 0 0
- joint jRightHip_roty: axis 0 0 1 -> 0 0 -1
- joint jRightHip_rotz: axis 0 1 0 -> 0 -1 0
- joint jRightKnee_roty: axis 0 1 0 -> 0 0 -1
- joint jRightKnee_rotz: axis 0 0 1 -> 0 -1 0
- joint jRightShoulder_rotx: origin xyz=0 0 0 rpy=0 0 0 -> xyz=0 0 0 rpy=1.5 0 0
- joint jRightShoulder_roty: axis 0 1 0 -> 0 0 1
- joint jRightShoulder_rotz: axis 0 0 1 -> 0 -1 0
- joint jRightWrist_rotz: axis 0 0 1 -> 0 -1 0
