Commit message: 🎮 Update ZJUHumanoid model

File: rofunc/simulator/assets/urdf/zju_humanoid/urdf/zju_humanoid.urdf (robot description, URDF)
Before this commit: robot 3N2-JUNE, 32 links, 31 joints
Links:
- link ASTRAGALUS_L: mass 25.9304036556032 -> 2.59; geometry visual mesh filename=../low_meshes/ASTRAGALUS_L.STL
- link ASTRAGALUS_R: mass 25.9304036556032 -> 2.59; geometry visual mesh filename=../low_meshes/ASTRAGALUS_R.STL
- link FOOT_L: mass 25.9304036556032 -> 2.59
- link FOOT_R: mass 25.9304036556032 -> 2.59
- link FOREARM_L: mass 25.9304036556032 -> 2.59
- link FOREARM_R: mass 25.9304036556032 -> 2.59
- link HAND_L: mass 25.9304036556032 -> 2.59; geometry visual mesh filename=../low_meshes/HAND_L.STL
- link HAND_R: mass 25.9304036556032 -> 2.59; geometry visual mesh filename=../low_meshes/HAND_R.STL
- link HEAD: mass 25.9304036556032 -> 2.59; geometry visual mesh filename=../low_meshes/HEAD.STL
- link ILIUM_L: mass 25.9304036556032 -> 2.59; geometry visual mesh filename=../low_meshes/ILIUM_L.STL
- link ILIUM_R: mass 25.9304036556032 -> 2.59; geometry visual mesh filename=../low_meshes/ILIUM_R.STL
- link ISCHIUM_L: mass 25.9304036556032 -> 2.59; geometry visual mesh filename=../low_meshes/ISCHIUM_L.STL
- link ISCHIUM_R: mass 25.9304036556032 -> 2.59; geometry visual mesh filename=../low_meshes/ISCHIUM_R.STL
- link NECK: mass 25.9304036556032 -> 2.59
- link SACRUM: mass 25.9304036556032 -> 2.59; geometry visual mesh filename=../low_meshes/SACRUM.STL
- link SCAPULA_L: mass 25.9304036556032 -> 2.59
- link SCAPULA_R: mass 25.9304036556032 -> 2.59
- link SHANK_L: mass 25.9304036556032 -> 2.59; geometry visual mesh filename=../low_meshes/SHANK_L.STL
- link SHANK_R: mass 25.9304036556032 -> 2.59; geometry visual mesh filename=../low_meshes/SHANK_R.STL
- link SHOULDER_L: mass 25.9304036556032 -> 2.59
- link SHOULDER_R: mass 25.9304036556032 -> 2.59
- link THIGH_L: mass 25.9304036556032 -> 2.59
- link THIGH_R: mass 25.9304036556032 -> 2.59
- link TIPTOE_Z_L: mass 6.67588438887831E-08 -> 2.59
- link TIPTOE_Z_R: mass 6.67588438887831E-08 -> 2.59
- link TORSO: mass 25.9304036556032 -> 2.59
- link UPPERARM_L: mass 25.9304036556032 -> 2.59
- link UPPERARM_R: mass 25.9304036556032 -> 2.59
- link WRIST_REVOLUTE_L: mass 25.9304036556032 -> 2.59
- link WRIST_REVOLUTE_R: mass 25.9304036556032 -> 2.59
- link WRIST_UPDOWN_L: mass 25.9304036556032 -> 2.59
- link WRIST_UPDOWN_R: mass 25.9304036556032 -> 2.59
Joints:
- joint Elbow_L: axis 0 -1 0 -> 0 1 0
- joint Hip_Y_L: axis 0 -1 0 -> 0 1 0
- joint Knee_L: axis 0 -1 0 -> 0 1 0
- joint Shoulder_Y_L: axis 0 1 0 -> 0 -1 0
