Commit message: 🎮 ZJUHumanoid pretrain amp5 OK!!!

File: rofunc/simulator/assets/urdf/zju_humanoid/urdf/zju_humanoid_new_inertia.urdf (robot description, URDF)
Before this commit: robot 3N2-JUNE, 32 links, 31 joints
Links:
- removed link TIPTOE_Z_L
- removed link TIPTOE_Z_R
Joints:
- removed joint Tiptoe_Z_L
- removed joint Tiptoe_Z_R
